File: Electronica de Potencia/TP's/TPN2/PCB/[PCB] Tp2_kicad/dimmer/dimmer.sch (KiCad schematic (older format))
At the start: 20 parts, among them J1 Conn_01x02, J2 Conn_01x02, Q1 2N2647, Q2 TIC106

Commit message: Rediseño dimmer
Parts:
- added TP1, TP2: TestPoint_2Pole, lib_fp:PinSocket_1x02_P2.54mm_Vertical, symbol dimmer_sch:Connector_TestPoint_2Pole
- C1: symbol dimmer_sch:Device_C -> dimmer_sch:dimmer-rescue_Device_C-dimmer_sch
- D1: symbol dimmer_sch:Diode_1N4007 -> dimmer_sch:1N4007
- DZ1: symbol dimmer_sch:Diode_1N47xxA -> dimmer_sch:dimmer-rescue_Diode_1N47xxA-dimmer_sch
- F1: symbol dimmer_sch:Device_Fuse -> dimmer_sch:dimmer-rescue_Device_Fuse-dimmer_sch
- G1: symbol dimmer-rescue:LOGO-logo -> dimmer_sch:dimmer-rescue_LOGO-logo
- J1: value Conn_01x02 -> Vin; symbol dimmer_sch:Connector_Generic_Conn_01x02 -> dimmer_sch:dimmer-rescue_Connector_Generic_Conn_01x02-dimmer_sch
- J2: value Conn_01x02 -> Vout; symbol dimmer_sch:Connector_Generic_Conn_01x02 -> dimmer_sch:dimmer-rescue_Connector_Generic_Conn_01x02-dimmer_sch
- Q1: symbol dimmer_sch:2N2647 -> dimmer_sch:dimmer_sch_2N2647
- Q2: symbol dimmer_sch:Triac_Thyristor_TIC106 -> dimmer_sch:dimmer-rescue_Triac_Thyristor_TIC106-dimmer_sch
- R1, R3, R4, R5: symbol dimmer_sch:Device_R_US -> dimmer_sch:dimmer-rescue_Device_R_US-dimmer_sch
- R2: symbol dimmer_sch:Device_R_POT -> dimmer_sch:dimmer-rescue_Device_R_POT-dimmer_sch
- RV1, RV2: symbol dimmer_sch:Device_R_POT_TRIM -> dimmer_sch:dimmer-rescue_Device_R_POT_TRIM-dimmer_sch
Connections:
- net Vref-: now reaches C1.2, D1.2 (A), D2.2 (A), DZ1.2 (A), Q2.1 (K), R4.2, RV2.3
- net Vref-: now also TP1.2
- net Load+: now reaches F1.2, J2.2 (Pin_2)
- net Load+: now also TP2.1
- net Load-: now reaches D1.1 (K), D3.2 (A), J2.1 (Pin_1)
- net Load-: now also TP2.2
- net Vref+: now reaches D5.2 (A), R2.2
- net Vref+: now also TP1.1
Other:
- moved on the sheet: G1, R4
Changed lines of the file:
@@
 $EndComp
 Wire Wire Line
-	3050 4700 3050 4550
+	3050 4700 3050 4650
 Wire Wire Line
 	3050 3600 3050 3000
@@
 	4150 3000 3750 3000
 $Comp
-L dimmer_sch:Diode_1N4007 D1
+L dimmer_sch:1N4007 D1
 U 1 1 5CB41FF5
 P 4500 3250
@@
 	4500 4050 4500 3950
 Wire Wire Line
-	4500 4350 4500 4550
-Wire Wire Line
-	4500 4550 3050 4550
-Connection ~ 3050 4550
-Wire Wire Line
-	3050 4550 3050 3700
+	4500 4350 4500 4650
+Wire Wire Line
+	4500 4650 3050 4650
+Connection ~ 3050 4650
+Wire Wire Line
+	3050 4650 3050 3700
 $Comp
 L dimmer_sch:1N4007 D3
@@
 	5050 4050 5050 3800
 Wire Wire Line
-	5050 4350 5050 4550
-Wire Wire Line
-	5050 4550 4500 4550
-Connection ~ 4500 4550
-$Comp
-L dimmer_sch:Device_R_US R1
+	5050 4350 5050 4650
+Wire Wire Line
+	5050 4650 4500 4650
+Connection ~ 4500 4650
+$Comp
+L dimmer_sch:dimmer-rescue_Device_R_US-dimmer_sch R1
 U 1 1 5CB46F56
 P 5800 3250
@@
 	5800 3100 5800 3000
 Wire Wire Line
-	5500 4550 5500 3950
+	5500 4650 5500 3950
 Wire Wire Line
 	5500 3950 4500 3950
@@
 	5500 3000 5800 3000
 $Comp
-L dimmer_sch:Device_R_POT R2
+L dimmer_sch:dimmer-rescue_Device_R_POT-dimmer_sch R2
 U 1 1 5CB4BC13
 P 6350 4000
@@
 $EndComp
 $Comp
-L dimmer_sch:Device_R_US R5
+L dimmer_sch:dimmer-rescue_Device_R_US-dimmer_sch R5
 U 1 1 5CB4E3DE
 P 7150 3650
@@
 	6350 4150 6350 4200
 Wire Wire Line
-	6500 4000 6700 4000
+	6500 4000 6650 4000
 Wire Wire Line
 	7150 3800 7150 4000
@@
 Connection ~ 5800 3000
 $Comp
-L dimmer_sch:Device_C C1
+L dimmer_sch:dimmer-rescue_Device_C-dimmer_sch C1
 U 1 1 5CB50EF3
 P 7150 4300
@@
 Connection ~ 7150 4000
 Wire Wire Line
-	7150 4450 7150 4550
-Wire Wire Line
-	7150 4550 6350 4550
-Connection ~ 6350 4550
-$Comp
-L dimmer_sch:Device_R_US R3
+	7150 4450 7150 4650
+Wire Wire Line
+	7150 4650 6650 4650
+Connection ~ 6350 4650
+$Comp
+L dimmer_sch:dimmer-rescue_Device_R_US-dimmer_sch R3
 U 1 1 5CB539F8
 P 7700 3650
@@
 Connection ~ 6350 3450
 $Comp
-L dimmer_sch:Device_R_US R4
+L dimmer_sch:dimmer-rescue_Device_R_US-dimmer_sch R4
 U 1 1 5CB56B3A
-P 7700 4400
-F 0 "R4" H 7768 4446 50  0000 L CNN
-F 1 "82" H 7768 4355 50  0000 L CNN
-F 2 "lib_fp:R_Axial_DIN0207_L6.3mm_D2.5mm_P10.16mm_Horizontal" V 7740 4390 50  0001 C CNN
-F 3 "~" H 7700 4400 50  0001 C CNN
-	1    7700 4400
-	1    0    0    -1
-$EndComp
-Connection ~ 7150 4550
+P 7700 4450
+F 0 "R4" H 7768 4496 50  0000 L CNN
+F 1 "82" H 7768 4405 50  0000 L CNN
+F 2 "lib_fp:R_Axial_DIN0207_L6.3mm_D2.5mm_P10.16mm_Horizontal" V 7740 4440 50  0001 C CNN
+F 3 "~" H 7700 4450 50  0001 C CNN
+	1    7700 4450
+	1    0    0    -1
+$EndComp
+Connection ~ 7150 4650
 Wire Wire Line
 	7700 4250 7700 4200
 $Comp
-L dimmer_sch:Triac_Thyristor_TIC106 Q2
+L dimmer_sch:dimmer-rescue_Triac_Thyristor_TIC106-dimmer_sch Q2
 U 1 1 5CB5862B
 P 8350 4150
@@
 	8200 4250 7700 4250
 Wire Wire Line
-	8350 4300 8350 4550
-$Comp
-L dimmer_sch:Device_R_POT_TRIM RV1
+	8350 4300 8350 4650
+$Comp
+L dimmer_sch:dimmer-rescue_Device_R_POT_TRIM-dimmer_sch RV1
 U 1 1 5CB49215
 P 6350 3650
@@
 	6500 3450 7700 3450
 $Comp
-L dimmer_sch:Device_R_POT_TRIM RV2
+L dimmer_sch:dimmer-rescue_Device_R_POT_TRIM-dimmer_sch RV2
 U 1 1 5CB4C207
 P 6350 4350
@@
 $EndComp
 Wire Wire Line
-	6350 4500 6350 4550
+	6350 4500 6350 4650
 Wire Wire Line
 	6500 4350 6500 4200
@@
 	6500 4200 6350 4200
 $Comp
-L dimmer_sch:Device_Fuse F1
+L dimmer_sch:dimmer-rescue_Device_Fuse-dimmer_sch F1
 U 1 1 5CB3DBB7
 P 3600 3000
@@
 $EndComp
 $Comp
-L dimmer_sch:power_GND #PWR01
+L dimmer_sch:dimmer-rescue_power_GND-dimmer_sch #PWR01
 U 1 1 5CB3F7B4
 P 3050 4700
@@
 $EndComp
 $Comp
-L dimmer_sch:Connector_Generic_Conn_01x02 J1
+L dimmer_sch:dimmer-rescue_Connector_Generic_Conn_01x02-dimmer_sch J1
 U 1 1 5CB3ADF7
 P 3250 3600
 F 0 "J1" H 3168 3275 50  0000 C CNN
-F 1 "Conn_01x02" H 3168 3366 50  0000 C CNN
+F 1 "Vin" H 3168 3366 50  0000 C CNN
 F 2 "lib_fp:TerminalBlock_bornier-2_P5.08mm" H 3250 3600 50  0001 C CNN
 F 3 "~" H 3250 3600 50  0001 C CNN
@@
 $EndComp
 Wire Wire Line
-	7150 4550 7700 4550
-$Comp
-L dimmer_sch:Connector_Generic_Conn_01x02 J2
+	7150 4650 7700 4650
+$Comp
+L dimmer_sch:dimmer-rescue_Connector_Generic_Conn_01x02-dimmer_sch J2
 U 1 1 5CB3E0B6
 P 4250 3200
 F 0 "J2" V 4214 3012 50  0000 R CNN
-F 1 "Conn_01x02" V 4123 3012 50  0000 R CNN
+F 1 "Vout" V 4123 3012 50  0000 R CNN
 F 2 "lib_fp:TerminalBlock_bornier-2_P5.08mm" H 4250 3200 50  0001 C CNN
 F 3 "~" H 4250 3200 50  0001 C CNN
@@
 $EndComp
 $Comp
-L dimmer-rescue:LOGO-logo G1
+L dimmer_sch:dimmer-rescue_LOGO-logo G1
 U 1 1 5CB4E2BD
-P 3500 4800
-F 0 "G1" H 3575 4853 60  0000 L CNN
-F 1 "LOGO" H 3575 4747 60  0000 L CNN
-F 2 "lib_fp:logo_utn_fsilk_small" H 3500 4800 50  0001 C CNN
-F 3 "" H 3500 4800 50  0001 C CNN
-	1    3500 4800
+P 3700 4350
+F 0 "G1" H 3775 4403 60  0000 L CNN
+F 1 "LOGO" H 3775 4297 60  0000 L CNN
+F 2 "lib_fp:logo_utn_fsilk_small" H 3700 4350 50  0001 C CNN
+F 3 "" H 3700 4350 50  0001 C CNN
+	1    3700 4350
 	1    0    0    -1
 $EndComp
@@
 	8350 4000 8350 3000
 $Comp
-L dimmer_sch:2N2647 Q1
+L dimmer_sch:dimmer_sch_2N2647 Q1
 U 1 1 5CB52F99
 P 7600 4000
@@
 $EndComp
 Wire Wire Line
-	5500 4550 5800 4550
-$Comp
-L dimmer_sch:Diode_1N47xxA DZ1
+	5500 4650 5800 4650
+$Comp
+L dimmer_sch:dimmer-rescue_Diode_1N47xxA-dimmer_sch DZ1
 U 1 1 5CB5BBFF
 P 5800 4000
@@
 Connection ~ 5800 3450
 Wire Wire Line
-	5800 4150 5800 4550
-Connection ~ 5800 4550
-Wire Wire Line
-	5800 4550 6350 4550
-Connection ~ 7700 4550
-Wire Wire Line
-	7700 4550 8350 4550
+	5800 4150 5800 4650
+Connection ~ 5800 4650
+Wire Wire Line
+	5800 4650 6350 4650
+Wire Wire Line
+	7700 4650 8350 4650
+Wire Wire Line
+	7700 4300 7700 4250
+Connection ~ 7700 4250
+Wire Wire Line
+	7700 4600 7700 4650
+Connection ~ 7700 4650
+Wire Wire Line
+	6650 3800 6650 4000
+Connection ~ 6650 4000
+Wire Wire Line
+	6650 4000 6700 4000
+Text Label 8900 3250 2    50   ~ 0
+Vref+
+Text Label 9400 3250 0    50   ~ 0
+Vref-
+Text Label 6650 3800 2    50   ~ 0
+Vref+
+Text Label 6650 4550 2    50   ~ 0
+Vref-
+Wire Wire Line
+	6650 4550 6650 4650
+Connection ~ 6650 4650
+Wire Wire Line
+	6650 4650 6350 4650
+Text Label 9950 3250 2    50   ~ 0
+Load+
+Text Label 10450 3250 0    50   ~ 0
+Load-
+Text Label 4250 2850 1    50   ~ 0
+Load-
+Wire Wire Line
+	4150 2850 4150 3000
+Text Label 4150 2850 1    50   ~ 0
+Load+
+Wire Wire Line
+	4250 2850 4250 3000
+$Comp
+L dimmer_sch:Connector_TestPoint_2Pole TP1
+U 1 1 5CC28AAA
+P 9150 3250
+F 0 "TP1" H 9150 3445 50  0000 C CNN
+F 1 "TestPoint_2Pole" H 9150 3354 50  0000 C CNN
+F 2 "lib_fp:PinSocket_1x02_P2.54mm_Vertical" H 9150 3250 50  0001 C CNN
+F 3 "~" H 9150 3250 50  0001 C CNN
+	1    9150 3250
+	1    0    0    -1
+$EndComp
+Wire Wire Line
+	8900 3250 8950 3250
+Wire Wire Line
+	9400 3250 9350 3250
+$Comp
+L dimmer_sch:Connector_TestPoint_2Pole TP2
+U 1 1 5CC3044A
+P 10200 3250
+F 0 "TP2" H 10200 3445 50  0000 C CNN
+F 1 "TestPoint_2Pole" H 10200 3354 50  0000 C CNN
+F 2 "lib_fp:PinSocket_1x02_P2.54mm_Vertical" H 10200 3250 50  0001 C CNN
+F 3 "~" H 10200 3250 50  0001 C CNN
+	1    10200 3250
+	1    0    0    -1
+$EndComp
+Wire Wire Line
+	9950 3250 10000 3250
+Wire Wire Line
+	10450 3250 10400 3250
 $EndSCHEMATC
