File: Tecnologia Electronica/Informe/Kicad [Circuito]/Circuito Tecnologia/Circuito Tecnologia.sch (KiCad schematic (older format))
At the start: 17 parts, among them J1 Conn_01x02, J2 Conn_01x03, K1 DIPxx-1Cxx-51x, Q1 2N2219, U1 L7805, U2 PIC16F886-IP, U3 SFH617A-1X001, Y1 Crystal

Commit message: Agrego cosas de tecnologia
Parts:
- 0,1uF: renamed from C3; symbol Device:C_Small -> Circuito-Tecnologia-rescue:C_Small-Device
- 0,1uF: renamed from C4; symbol Device:C_Small -> Circuito-Tecnologia-rescue:C_Small-Device
- 0,1uF: renamed from C2; symbol Device:C_Small -> Circuito-Tecnologia-rescue:C_Small-Device
- 0,33uF: renamed from C1; symbol Device:C_Small -> Circuito-Tecnologia-rescue:C_Small-Device
- 10k: renamed from R2; symbol Device:R_US -> Circuito-Tecnologia-rescue:R_US-Device
- 1k: renamed from R1; symbol Device:R_US -> Circuito-Tecnologia-rescue:R_US-Device
- D1: symbol Diode:1N4148 -> Circuito-Tecnologia-rescue:1N4148-Diode
- D2: symbol Device:LED -> Circuito-Tecnologia-rescue:LED-Device
- J1: symbol Connector_Generic:Conn_01x02 -> Circuito-Tecnologia-rescue:Conn_01x02-Connector_Generic
- J2: symbol Connector_Generic:Conn_01x03 -> Circuito-Tecnologia-rescue:Conn_01x03-Connector_Generic
- K1: symbol Relay:DIPxx-1Cxx-51x -> Circuito-Tecnologia-rescue:DIPxx-1Cxx-51x-Relay
- PC817C: renamed from U3; symbol Isolator:SFH617A-1X001 -> Circuito-Tecnologia-rescue:SFH617A-1X001-Isolator
- Q1: value 2N2219 -> MMBT5551; symbol Transistor_BJT:2N2219 -> Circuito-Tecnologia-rescue:2N2219-Transistor_BJT
- R3: value 100 -> 510; symbol Device:R_US -> Circuito-Tecnologia-rescue:R_US-Device
- U1: symbol Regulator_Linear:L7805 -> Circuito-Tecnologia-rescue:L7805-Regulator_Linear
- U2: symbol MCU_Microchip_PIC16:PIC16F886-IP -> Circuito-Tecnologia-rescue:PIC16F886-IP-MCU_Microchip_PIC16
- Y1: symbol Device:Crystal -> Circuito-Tecnologia-rescue:Crystal-Device
Connections:
- net +5V: now also K1.6
Changed lines of the file:
@@
 EESchema Schematic File Version 4
+LIBS:Circuito Tecnologia-cache
 EELAYER 29 0
 EELAYER END
@@
 $EndDescr
 $Comp
-L MCU_Microchip_PIC16:PIC16F886-IP U2
+L Circuito-Tecnologia-rescue:PIC16F886-IP-MCU_Microchip_PIC16 U2
 U 1 1 5CBA8C4A
 P 4700 3400
@@
 $EndComp
 $Comp
-L Device:Crystal Y1
+L Circuito-Tecnologia-rescue:Crystal-Device Y1
 U 1 1 5CBA985E
 P 6400 3250
@@
 	6200 3400 6400 3400
 $Comp
-L Device:C_Small C3
+L Circuito-Tecnologia-rescue:C_Small-Device 0,1uF
 U 1 1 5CBB10D6
 P 6700 3100
-F 0 "C3" V 6563 3100 50  0000 C CNN
+F 0 "0,1uF" V 6563 3100 50  0000 C CNN
 F 1 "0.1uF" V 6562 3100 50  0001 C CNN
 F 2 "" H 6700 3100 50  0001 C CNN
@@
 $EndComp
 $Comp
-L Device:C_Small C4
+L Circuito-Tecnologia-rescue:C_Small-Device 0,1uF
 U 1 1 5CBB1C68
 P 6700 3400
-F 0 "C4" V 6850 3400 50  0000 C CNN
+F 0 "0,1uF" V 6850 3400 50  0000 C CNN
 F 1 "0.1uF" V 6900 3400 50  0001 C CNN
 F 2 "" H 6700 3400 50  0001 C CNN
@@
 	6900 3100 6800 3100
 $Comp
-L power:GND #PWR0101
+L Circuito-Tecnologia-rescue:GND-power #PWR0101
 U 1 1 5CBB2EC2
 P 7050 3300
@@
 	6900 3250 6900 3100
 $Comp
-L Regulator_Linear:L7805 U1
+L Circuito-Tecnologia-rescue:L7805-Regulator_Linear U1
 U 1 1 5CBB4893
 P 2550 2600
@@
 $EndComp
 $Comp
-L Device:C_Small C2
+L Circuito-Tecnologia-rescue:C_Small-Device 0,1uF
 U 1 1 5CBB5A7D
 P 3000 2700
-F 0 "C2" H 2908 2700 50  0000 R CNN
+F 0 "0,1uF" H 2908 2700 50  0000 R CNN
 F 1 "0.1 uF" H 2908 2745 50  0001 R CNN
 F 2 "" H 3000 2700 50  0001 C CNN
@@
 $EndComp
 $Comp
-L Device:C_Small C1
+L Circuito-Tecnologia-rescue:C_Small-Device 0,33uF
 U 1 1 5CBB63B6
 P 2100 2700
-F 0 "C1" H 1900 2700 50  0000 L CNN
+F 0 "0,33uF" H 1750 2700 50  0000 L CNN
 F 1 "0.33uF" H 1700 2650 50  0001 L CNN
 F 2 "" H 2100 2700 50  0001 C CNN
@@
 	3000 2600 2850 2600
 $Comp
-L power:GND #PWR0102
+L Circuito-Tecnologia-rescue:GND-power #PWR0102
 U 1 1 5CBBA8C3
 P 4750 4600
@@
 Connection ~ 4750 4600
 $Comp
-L Isolator:SFH617A-1X001 U3
+L Circuito-Tecnologia-rescue:SFH617A-1X001-Isolator PC817C
 U 1 1 5CBBECD8
 P 7650 4100
-F 0 "U3" H 7650 4333 50  0000 C CNN
+F 0 "PC817C" H 7650 4333 50  0000 C CNN
 F 1 "SFH617A-1X001" H 7650 4334 50  0001 C CNN
 F 2 "Package_DIP:DIP-4_W7.62mm" H 7450 3900 50  0001 L CIN
@@
 	3250 2600 3400 2600
 $Comp
-L Relay:DIPxx-1Cxx-51x K1
+L Circuito-Tecnologia-rescue:DIPxx-1Cxx-51x-Relay K1
 U 1 1 5CBD5167
 P 8950 2950
@@
 $EndComp
 $Comp
-L Connector_Generic:Conn_01x02 J1
+L Circuito-Tecnologia-rescue:Conn_01x02-Connector_Generic J1
 U 1 1 5CBDFD63
 P 1350 2700
@@
 Connection ~ 2100 2600
 $Comp
-L power:GND #PWR0105
+L Circuito-Tecnologia-rescue:GND-power #PWR0105
 U 1 1 5CBE15B9
 P 1650 2800
@@
 	1650 2700 1550 2700
 $Comp
-L Transistor_BJT:2N2219 Q1
+L Circuito-Tecnologia-rescue:2N2219-Transistor_BJT Q1
 U 1 1 5CBE48F2
 P 8650 4200
-F 0 "Q1" H 8840 4200 50  0000 L CNN
-F 1 "2N2219" H 8840 4155 50  0001 L CNN
+F 0 "Q1" H 8840 4200 50  0001 L CNN
+F 1 "MMBT5551" H 8840 4155 50  0000 L CNN
 F 2 "Package_TO_SOT_THT:TO-39-3" H 8850 4125 50  0001 L CIN
 F 3 "http://www.onsemi.com/pub_link/Collateral/2N2219-D.PDF" H 8650 4200 50  0001 L CNN
@@
 $EndComp
 $Comp
-L Device:R_US R3
+L Circuito-Tecnologia-rescue:R_US-Device R3
 U 1 1 5CBEACA4
 P 8200 4200
-F 0 "R3" V 8100 4200 50  0000 C CNN
-F 1 "100" V 8300 4200 50  0001 C CNN
+F 0 "R3" V 8100 4200 50  0001 C CNN
+F 1 "510" V 8300 4200 50  0000 C CNN
 F 2 "" V 8240 4190 50  0001 C CNN
 F 3 "~" H 8200 4200 50  0001 C CNN
@@
 $EndComp
 $Comp
-L Diode:1N4148 D1
+L Circuito-Tecnologia-rescue:1N4148-Diode D1
 U 1 1 5CBC1B51
 P 8350 3000
-F 0 "D1" H 8300 2900 50  0000 L CNN
-F 1 "1N4148" H 8200 3100 50  0001 L CNN
+F 0 "D1" H 8300 2900 50  0001 L CNN
+F 1 "1N4148" H 8200 3100 50  0000 L CNN
 F 2 "Diode_THT:D_DO-35_SOD27_P7.62mm_Horizontal" H 8350 2825 50  0001 C CNN
 F 3 "https://assets.nexperia.com/documents/data-sheet/1N4148_1N4448.pdf" H 8350 3000 50  0001 C CNN
@@
 $EndComp
 $Comp
-L power:GND #PWR01
+L Circuito-Tecnologia-rescue:GND-power #PWR01
 U 1 1 5CC06B8D
 P 8750 4500
@@
 Connection ~ 4700 2300
 $Comp
-L Connector_Generic:Conn_01x03 J2
+L Circuito-Tecnologia-rescue:Conn_01x03-Connector_Generic J2
 U 1 1 5CC0BC33
 P 10000 3000
@@
 	9650 3100 9800 3100
 $Comp
-L Device:LED D2
+L Circuito-Tecnologia-rescue:LED-Device D2
 U 1 1 5CC1A569
 P 6750 4200
@@
 	6900 4200 7350 4200
 $Comp
-L Device:R_US R1
+L Circuito-Tecnologia-rescue:R_US-Device 1k
 U 1 1 5CC23A41
 P 7300 3250
-F 0 "R1" H 7200 3250 50  0000 C CNN
+F 0 "1k" H 7200 3250 50  0000 C CNN
 F 1 "100" V 7400 3250 50  0001 C CNN
 F 2 "" V 7340 3240 50  0001 C CNN
@@
 	8350 2850 8350 2300
 Wire Wire Line
-	8350 2300 9050 2300
+	8350 2300 8750 2300
 Connection ~ 9050 2300
 Wire Wire Line
@@
 Connection ~ 8350 2300
 $Comp
-L power:+5V #PWR02
+L Circuito-Tecnologia-rescue:+5V-power #PWR02
 U 1 1 5CC3D910
 P 3250 2200
@@
 	6350 4200 6000 4200
 $Comp
-L Device:R_US R2
+L Circuito-Tecnologia-rescue:R_US-Device 10k
 U 1 1 5CC42B30
 P 6350 3900
-F 0 "R2" V 6250 3900 50  0000 C CNN
+F 0 "10k" V 6250 3900 50  0000 C CNN
 F 1 "100" V 6450 3900 50  0001 C CNN
 F 2 "" V 6390 3890 50  0001 C CNN
@@
 	2550 2950 2550 2900
 $Comp
-L power:GND #PWR?
+L Circuito-Tecnologia-rescue:GND-power #PWR?
 U 1 1 5CC481AD
 P 2550 2950
@@
 	6350 3750 6350 3700
 $Comp
-L power:+5V #PWR03
+L Circuito-Tecnologia-rescue:+5V-power #PWR03
 U 1 1 5CC3FA58
 P 6350 3700
@@
 	1    0    0    -1
 $EndComp
+Wire Wire Line
+	8750 2650 8750 2300
+Connection ~ 8750 2300
+Wire Wire Line
+	8750 2300 9050 2300
 $EndSCHEMATC
