File: Electronica Aplicada 3/TP's/TPN2/PCB/[PCB] Kicad/hartley/osciladores.kicad_pcb (KiCad board)
At the start: 2 copper layers, 45 parts, among them J1 Conn_01x01_Female, J2 Conn_01x01_Female, J3 Conn_01x01_Female, J4 Conn_01x01_Female, Q1 2N3904

Commit message: Agrego rediseño de Hartley (kicad)
Parts:
- removed the C1 at (50.8, 163.8)
- removed the C1 at (166.4, 81.3)
- removed the C1 at (48.3, 81.3)
- removed the C2 at (82.5, 138.4)
- removed the C2 at (198.1, 55.9)
- removed the C2 at (80.0, 55.9)
- removed the C3 at (114.3, 115.6)
- removed the C3 at (229.9, 33.0)
- removed the C3 at (111.8, 33.0)
- removed the J1 at (45.7, 123.2)
- removed the J1 at (161.3, 40.6)
- removed the J1 at (43.2, 40.6)
- removed the J2 at (39.4, 111.8)
- removed the J2 at (154.9, 29.2)
- removed the J2 at (36.8, 29.2)
- removed the J3 at (124.5, 154.9)
- removed the J3 at (240.0, 72.4)
- removed the J3 at (121.9, 72.4)
- removed the J4 at (110.5, 154.9)
- removed the J4 at (226.1, 72.4)
- removed the J4 at (108.0, 72.4)
- removed the L1 at (118.1, 142.2)
- removed the L1 at (233.7, 59.7)
- removed the L1 at (115.6, 59.7)
- removed the L2 at (83.8, 170.2)
- removed the L2 at (199.4, 87.6)
- removed the L2 at (81.3, 87.6)
- removed the Q1 at (63.5, 134.6)
- removed the Q1 at (179.1, 52.1)
- removed the Q1 at (61.0, 52.1)
- removed the R1 at (54.6, 113.0)
- removed the R1 at (170.2, 30.5)
- removed the R1 at (52.1, 30.5)
- removed the R2 at (45.7, 141.0)
- removed the R2 at (161.3, 58.4)
- removed the R2 at (43.2, 58.4)
- removed the R3 at (76.2, 113.0)
- removed the R3 at (191.8, 30.5)
- removed the R3 at (73.7, 30.5)
- removed R4 (x3): R, Resistors_THT:R_Box_L13.0mm_W4.0mm_P9.00mm
- removed the RV1 at (72.4, 148.6)
- removed the RV1 at (188.0, 66.0)
- removed the RV1 at (69.8, 66.0)
- added C1: C, Capacitor_THT:C_Disc_D5.0mm_W2.5mm_P5.00mm, F.Cu at (120.7, 170.3)
- added C1: C, Capacitor_THT:C_Disc_D5.0mm_W2.5mm_P5.00mm, F.Cu at (185.2, 84.0)
- added C1: C, Capacitor_THT:C_Disc_D5.0mm_W2.5mm_P5.00mm, F.Cu at (252.6, 83.9)
- added C1: C, Capacitor_THT:C_Disc_D5.0mm_W2.5mm_P5.00mm, F.Cu at (49.9, 83.7)
- added C1: C, Capacitor_THT:C_Disc_D5.0mm_W2.5mm_P5.00mm, F.Cu at (251.6, 34.2)
- added C1: C, Capacitor_THT:C_Disc_D5.0mm_W2.5mm_P5.00mm, F.Cu at (184.3, 34.3)
- added C1: C, Capacitor_THT:C_Disc_D5.0mm_W2.5mm_P5.00mm, F.Cu at (116.3, 33.9)
- added C1: C, Capacitor_THT:C_Disc_D5.0mm_W2.5mm_P5.00mm, F.Cu at (48.9, 34.1)
- added C1: C, Capacitor_THT:C_Disc_D5.0mm_W2.5mm_P5.00mm, F.Cu at (188.7, 170.8)
- added C1: C, Capacitor_THT:C_Disc_D5.0mm_W2.5mm_P5.00mm, F.Cu at (256.0, 170.6)
- added C1: C, Capacitor_THT:C_Disc_D5.0mm_W2.5mm_P5.00mm, F.Cu at (53.3, 170.5)
- added C1: C, Capacitor_THT:C_Disc_D5.0mm_W2.5mm_P5.00mm, F.Cu at (119.5, 129.1)
- added C1: C, Capacitor_THT:C_Disc_D5.0mm_W2.5mm_P5.00mm, F.Cu at (187.5, 129.5)
- added C1: C, Capacitor_THT:C_Disc_D5.0mm_W2.5mm_P5.00mm, F.Cu at (254.9, 129.3)
- added C1: C, Capacitor_THT:C_Disc_D5.0mm_W2.5mm_P5.00mm, F.Cu at (52.2, 129.2)
- added C1: C, Capacitor_THT:C_Disc_D5.0mm_W2.5mm_P5.00mm, F.Cu at (117.2, 83.6)
- added C2: C, Capacitor_THT:C_Disc_D7.5mm_W2.5mm_P5.00mm, F.Cu at (127.8, 165.6)
- added C2: C, Capacitor_THT:C_Disc_D7.5mm_W2.5mm_P5.00mm, F.Cu at (259.7, 79.2)
- added C2: C, Capacitor_THT:C_Disc_D7.5mm_W2.5mm_P5.00mm, F.Cu at (192.4, 79.3)
- added C2: C, Capacitor_THT:C_Disc_D7.5mm_W2.5mm_P5.00mm, F.Cu at (57.1, 79.0)
- added C2: C, Capacitor_THT:C_Disc_D7.5mm_W2.5mm_P5.00mm, F.Cu at (258.7, 29.5)
- added C2: C, Capacitor_THT:C_Disc_D7.5mm_W2.5mm_P5.00mm, F.Cu at (191.4, 29.6)
- added C2: C, Capacitor_THT:C_Disc_D7.5mm_W2.5mm_P5.00mm, F.Cu at (123.4, 29.2)
- added C2: C, Capacitor_THT:C_Disc_D7.5mm_W2.5mm_P5.00mm, F.Cu at (56.1, 29.4)
- added C2: C, Capacitor_THT:C_Disc_D7.5mm_W2.5mm_P5.00mm, F.Cu at (263.2, 165.9)
- added C2: C, Capacitor_THT:C_Disc_D7.5mm_W2.5mm_P5.00mm, F.Cu at (195.8, 166.1)
- added C2: C, Capacitor_THT:C_Disc_D7.5mm_W2.5mm_P5.00mm, F.Cu at (60.5, 165.8)
- added C2: C, Capacitor_THT:C_Disc_D7.5mm_W2.5mm_P5.00mm, F.Cu at (126.7, 124.4)
- added C2: C, Capacitor_THT:C_Disc_D7.5mm_W2.5mm_P5.00mm, F.Cu at (262.0, 124.6)
- added C2: C, Capacitor_THT:C_Disc_D7.5mm_W2.5mm_P5.00mm, F.Cu at (194.7, 124.8)
- added C2: C, Capacitor_THT:C_Disc_D7.5mm_W2.5mm_P5.00mm, F.Cu at (59.4, 124.5)
- added C2: C, Capacitor_THT:C_Disc_D7.5mm_W2.5mm_P5.00mm, F.Cu at (124.4, 78.9)
- added C3: C, Capacitor_THT:C_Disc_D7.5mm_W2.5mm_P5.00mm, F.Cu at (118.1, 165.6)
- added C3: C, Capacitor_THT:C_Disc_D7.5mm_W2.5mm_P5.00mm, F.Cu at (250.0, 79.2)
- added C3: C, Capacitor_THT:C_Disc_D7.5mm_W2.5mm_P5.00mm, F.Cu at (182.6, 79.3)
- added C3: C, Capacitor_THT:C_Disc_D7.5mm_W2.5mm_P5.00mm, F.Cu at (47.3, 79.0)
- added C3: C, Capacitor_THT:C_Disc_D7.5mm_W2.5mm_P5.00mm, F.Cu at (249.0, 29.5)
- added C3: C, Capacitor_THT:C_Disc_D7.5mm_W2.5mm_P5.00mm, F.Cu at (181.6, 29.6)
- added C3: C, Capacitor_THT:C_Disc_D7.5mm_W2.5mm_P5.00mm, F.Cu at (113.6, 29.2)
- added C3: C, Capacitor_THT:C_Disc_D7.5mm_W2.5mm_P5.00mm, F.Cu at (46.3, 29.4)
- added C3: C, Capacitor_THT:C_Disc_D7.5mm_W2.5mm_P5.00mm, F.Cu at (253.4, 165.9)
- added C3: C, Capacitor_THT:C_Disc_D7.5mm_W2.5mm_P5.00mm, F.Cu at (186.1, 166.1)
- added C3: C, Capacitor_THT:C_Disc_D7.5mm_W2.5mm_P5.00mm, F.Cu at (50.7, 165.8)
- added C3: C, Capacitor_THT:C_Disc_D7.5mm_W2.5mm_P5.00mm, F.Cu at (116.9, 124.4)
- added C3: C, Capacitor_THT:C_Disc_D7.5mm_W2.5mm_P5.00mm, F.Cu at (252.2, 124.6)
- added C3: C, Capacitor_THT:C_Disc_D7.5mm_W2.5mm_P5.00mm, F.Cu at (184.9, 124.8)
- added C3: C, Capacitor_THT:C_Disc_D7.5mm_W2.5mm_P5.00mm, F.Cu at (49.6, 124.5)
- added C3: C, Capacitor_THT:C_Disc_D7.5mm_W2.5mm_P5.00mm, F.Cu at (114.6, 78.9)
- added C4: C, Capacitor_THT:C_Disc_D7.5mm_W2.5mm_P5.00mm, F.Cu at (136.5, 169.3)
- added C4: C, Capacitor_THT:C_Disc_D7.5mm_W2.5mm_P5.00mm, F.Cu at (268.4, 82.9)
- added C4: C, Capacitor_THT:C_Disc_D7.5mm_W2.5mm_P5.00mm, F.Cu at (201.1, 83.0)
- added C4: C, Capacitor_THT:C_Disc_D7.5mm_W2.5mm_P5.00mm, F.Cu at (65.7, 82.7)
- added C4: C, Capacitor_THT:C_Disc_D7.5mm_W2.5mm_P5.00mm, F.Cu at (267.4, 33.2)
- added C4: C, Capacitor_THT:C_Disc_D7.5mm_W2.5mm_P5.00mm, F.Cu at (200.1, 33.3)
- added C4: C, Capacitor_THT:C_Disc_D7.5mm_W2.5mm_P5.00mm, F.Cu at (132.1, 32.9)
- added C4: C, Capacitor_THT:C_Disc_D7.5mm_W2.5mm_P5.00mm, F.Cu at (64.7, 33.0)
- added C4: C, Capacitor_THT:C_Disc_D7.5mm_W2.5mm_P5.00mm, F.Cu at (271.8, 169.6)
- added C4: C, Capacitor_THT:C_Disc_D7.5mm_W2.5mm_P5.00mm, F.Cu at (204.5, 169.7)
- added C4: C, Capacitor_THT:C_Disc_D7.5mm_W2.5mm_P5.00mm, F.Cu at (69.2, 169.5)
- added C4: C, Capacitor_THT:C_Disc_D7.5mm_W2.5mm_P5.00mm, F.Cu at (135.4, 128.0)
- added C4: C, Capacitor_THT:C_Disc_D7.5mm_W2.5mm_P5.00mm, F.Cu at (270.7, 128.3)
- added C4: C, Capacitor_THT:C_Disc_D7.5mm_W2.5mm_P5.00mm, F.Cu at (203.4, 128.5)
- added C4: C, Capacitor_THT:C_Disc_D7.5mm_W2.5mm_P5.00mm, F.Cu at (68.0, 128.2)
- added C4: C, Capacitor_THT:C_Disc_D7.5mm_W2.5mm_P5.00mm, F.Cu at (133.1, 82.6)
- added C5: C, Capacitor_THT:C_Disc_D7.5mm_W2.5mm_P5.00mm, F.Cu at (136.6, 165.8)
- added C5: C, Capacitor_THT:C_Disc_D7.5mm_W2.5mm_P5.00mm, F.Cu at (268.5, 79.3)
- added C5: C, Capacitor_THT:C_Disc_D7.5mm_W2.5mm_P5.00mm, F.Cu at (201.1, 79.5)
- added C5: C, Capacitor_THT:C_Disc_D7.5mm_W2.5mm_P5.00mm, F.Cu at (65.8, 79.2)
- added C5: C, Capacitor_THT:C_Disc_D7.5mm_W2.5mm_P5.00mm, F.Cu at (267.5, 29.6)
- added C5: C, Capacitor_THT:C_Disc_D7.5mm_W2.5mm_P5.00mm, F.Cu at (200.1, 29.8)
- added C5: C, Capacitor_THT:C_Disc_D7.5mm_W2.5mm_P5.00mm, F.Cu at (132.1, 29.3)
- added C5: C, Capacitor_THT:C_Disc_D7.5mm_W2.5mm_P5.00mm, F.Cu at (64.8, 29.5)
- added C5: C, Capacitor_THT:C_Disc_D7.5mm_W2.5mm_P5.00mm, F.Cu at (271.9, 166.0)
- added C5: C, Capacitor_THT:C_Disc_D7.5mm_W2.5mm_P5.00mm, F.Cu at (204.5, 166.2)
- added C5: C, Capacitor_THT:C_Disc_D7.5mm_W2.5mm_P5.00mm, F.Cu at (69.2, 165.9)
- added C5: C, Capacitor_THT:C_Disc_D7.5mm_W2.5mm_P5.00mm, F.Cu at (135.4, 124.5)
- added C5: C, Capacitor_THT:C_Disc_D7.5mm_W2.5mm_P5.00mm, F.Cu at (270.7, 124.8)
- added C5: C, Capacitor_THT:C_Disc_D7.5mm_W2.5mm_P5.00mm, F.Cu at (203.4, 124.9)
- added C5: C, Capacitor_THT:C_Disc_D7.5mm_W2.5mm_P5.00mm, F.Cu at (68.1, 124.6)
- added C5: C, Capacitor_THT:C_Disc_D7.5mm_W2.5mm_P5.00mm, F.Cu at (133.1, 79.0)
- added C6: C, Capacitor_THT:C_Disc_D7.5mm_W2.5mm_P5.00mm, F.Cu at (199.6, 171.2)
- added C6: C, Capacitor_THT:C_Disc_D7.5mm_W2.5mm_P5.00mm, F.Cu at (263.5, 84.3)
- added C6: C, Capacitor_THT:C_Disc_D7.5mm_W2.5mm_P5.00mm, F.Cu at (128.2, 84.0)
- added C6: C, Capacitor_THT:C_Disc_D7.5mm_W2.5mm_P5.00mm, F.Cu at (60.8, 84.2)
- added C6: C, Capacitor_THT:C_Disc_D7.5mm_W2.5mm_P5.00mm, F.Cu at (262.5, 34.6)
- added C6: C, Capacitor_THT:C_Disc_D7.5mm_W2.5mm_P5.00mm, F.Cu at (195.2, 34.8)
- added C6: C, Capacitor_THT:C_Disc_D7.5mm_W2.5mm_P5.00mm, F.Cu at (127.2, 34.3)
- added C6: C, Capacitor_THT:C_Disc_D7.5mm_W2.5mm_P5.00mm, F.Cu at (59.8, 34.5)
- added C6: C, Capacitor_THT:C_Disc_D7.5mm_W2.5mm_P5.00mm, F.Cu at (266.9, 171.0)
- added C6: C, Capacitor_THT:C_Disc_D7.5mm_W2.5mm_P5.00mm, F.Cu at (131.6, 170.8)
- added C6: C, Capacitor_THT:C_Disc_D7.5mm_W2.5mm_P5.00mm, F.Cu at (64.3, 170.9)
- added C6: C, Capacitor_THT:C_Disc_D7.5mm_W2.5mm_P5.00mm, F.Cu at (198.5, 129.9)
- added C6: C, Capacitor_THT:C_Disc_D7.5mm_W2.5mm_P5.00mm, F.Cu at (265.8, 129.8)
- added C6: C, Capacitor_THT:C_Disc_D7.5mm_W2.5mm_P5.00mm, F.Cu at (130.5, 129.5)
- added C6: C, Capacitor_THT:C_Disc_D7.5mm_W2.5mm_P5.00mm, F.Cu at (63.1, 129.6)
- added C6: C, Capacitor_THT:C_Disc_D7.5mm_W2.5mm_P5.00mm, F.Cu at (196.2, 84.5)
- added J1: Conn_01x01_Female, Connector_PinHeader_2.54mm:PinHeader_1x01_P2.54mm_Horizontal, F.Cu at (93.5, 166.4)
- added J1: Conn_01x01_Female, Connector_PinHeader_2.54mm:PinHeader_1x01_P2.54mm_Horizontal, F.Cu at (225.5, 79.9)
- added J1: Conn_01x01_Female, Connector_PinHeader_2.54mm:PinHeader_1x01_P2.54mm_Horizontal, F.Cu at (158.1, 80.1)
- added J1: Conn_01x01_Female, Connector_PinHeader_2.54mm:PinHeader_1x01_P2.54mm_Horizontal, F.Cu at (22.8, 79.8)
- added J1: Conn_01x01_Female, Connector_PinHeader_2.54mm:PinHeader_1x01_P2.54mm_Horizontal, F.Cu at (224.5, 30.2)
- added J1: Conn_01x01_Female, Connector_PinHeader_2.54mm:PinHeader_1x01_P2.54mm_Horizontal, F.Cu at (157.1, 30.4)
- added J1: Conn_01x01_Female, Connector_PinHeader_2.54mm:PinHeader_1x01_P2.54mm_Horizontal, F.Cu at (89.1, 29.9)
- added J1: Conn_01x01_Female, Connector_PinHeader_2.54mm:PinHeader_1x01_P2.54mm_Horizontal, F.Cu at (21.8, 30.1)
- added J1: Conn_01x01_Female, Connector_PinHeader_2.54mm:PinHeader_1x01_P2.54mm_Horizontal, F.Cu at (228.9, 166.6)
- added J1: Conn_01x01_Female, Connector_PinHeader_2.54mm:PinHeader_1x01_P2.54mm_Horizontal, F.Cu at (161.5, 166.8)
- added J1: Conn_01x01_Female, Connector_PinHeader_2.54mm:PinHeader_1x01_P2.54mm_Horizontal, F.Cu at (26.2, 166.5)
- added J1: Conn_01x01_Female, Connector_PinHeader_2.54mm:PinHeader_1x01_P2.54mm_Horizontal, F.Cu at (92.4, 125.1)
- added J1: Conn_01x01_Female, Connector_PinHeader_2.54mm:PinHeader_1x01_P2.54mm_Horizontal, F.Cu at (227.7, 125.4)
- added J1: Conn_01x01_Female, Connector_PinHeader_2.54mm:PinHeader_1x01_P2.54mm_Horizontal, F.Cu at (160.4, 125.5)
- added J1: Conn_01x01_Female, Connector_PinHeader_2.54mm:PinHeader_1x01_P2.54mm_Horizontal, F.Cu at (25.1, 125.2)
- added J1: Conn_01x01_Female, Connector_PinHeader_2.54mm:PinHeader_1x01_P2.54mm_Horizontal, F.Cu at (90.1, 79.6)
- added J2: Conn_01x01_Female, Connector_PinHeader_2.54mm:PinHeader_1x01_P2.54mm_Horizontal, F.Cu at (93.1, 182.4)
- added J2: Conn_01x01_Female, Connector_PinHeader_2.54mm:PinHeader_1x01_P2.54mm_Horizontal, F.Cu at (225.0, 95.9)
- added J2: Conn_01x01_Female, Connector_PinHeader_2.54mm:PinHeader_1x01_P2.54mm_Horizontal, F.Cu at (157.7, 96.1)
- added J2: Conn_01x01_Female, Connector_PinHeader_2.54mm:PinHeader_1x01_P2.54mm_Horizontal, F.Cu at (22.4, 95.8)
- added J2: Conn_01x01_Female, Connector_PinHeader_2.54mm:PinHeader_1x01_P2.54mm_Horizontal, F.Cu at (224.0, 46.3)
- added J2: Conn_01x01_Female, Connector_PinHeader_2.54mm:PinHeader_1x01_P2.54mm_Horizontal, F.Cu at (156.7, 46.4)
- added J2: Conn_01x01_Female, Connector_PinHeader_2.54mm:PinHeader_1x01_P2.54mm_Horizontal, F.Cu at (88.7, 46.0)
- added J2: Conn_01x01_Female, Connector_PinHeader_2.54mm:PinHeader_1x01_P2.54mm_Horizontal, F.Cu at (21.4, 46.1)
- added J2: Conn_01x01_Female, Connector_PinHeader_2.54mm:PinHeader_1x01_P2.54mm_Horizontal, F.Cu at (228.4, 182.7)
- added J2: Conn_01x01_Female, Connector_PinHeader_2.54mm:PinHeader_1x01_P2.54mm_Horizontal, F.Cu at (161.1, 182.8)
- added J2: Conn_01x01_Female, Connector_PinHeader_2.54mm:PinHeader_1x01_P2.54mm_Horizontal, F.Cu at (25.8, 182.5)
- added J2: Conn_01x01_Female, Connector_PinHeader_2.54mm:PinHeader_1x01_P2.54mm_Horizontal, F.Cu at (92.0, 141.1)
- added J2: Conn_01x01_Female, Connector_PinHeader_2.54mm:PinHeader_1x01_P2.54mm_Horizontal, F.Cu at (227.3, 141.4)
- added J2: Conn_01x01_Female, Connector_PinHeader_2.54mm:PinHeader_1x01_P2.54mm_Horizontal, F.Cu at (160.0, 141.6)
- added J2: Conn_01x01_Female, Connector_PinHeader_2.54mm:PinHeader_1x01_P2.54mm_Horizontal, F.Cu at (24.6, 141.3)
- added J2: Conn_01x01_Female, Connector_PinHeader_2.54mm:PinHeader_1x01_P2.54mm_Horizontal, F.Cu at (89.7, 95.7)
- added J3: Conn_01x01_Female, Connector_PinHeader_2.54mm:PinHeader_1x01_P2.54mm_Horizontal, F.Cu at (276.2, 173.5)
- added J3: Conn_01x01_Female, Connector_PinHeader_2.54mm:PinHeader_1x01_P2.54mm_Horizontal, F.Cu at (205.4, 86.9)
- added J3: Conn_01x01_Female, Connector_PinHeader_2.54mm:PinHeader_1x01_P2.54mm_Horizontal, F.Cu at (137.4, 86.5)
- added J3: Conn_01x01_Female, Connector_PinHeader_2.54mm:PinHeader_1x01_P2.54mm_Horizontal, F.Cu at (70.1, 86.7)
- added J3: Conn_01x01_Female, Connector_PinHeader_2.54mm:PinHeader_1x01_P2.54mm_Horizontal, F.Cu at (271.8, 37.1)
- added J3: Conn_01x01_Female, Connector_PinHeader_2.54mm:PinHeader_1x01_P2.54mm_Horizontal, F.Cu at (204.4, 37.3)
- added J3: Conn_01x01_Female, Connector_PinHeader_2.54mm:PinHeader_1x01_P2.54mm_Horizontal, F.Cu at (136.4, 36.8)
- added J3: Conn_01x01_Female, Connector_PinHeader_2.54mm:PinHeader_1x01_P2.54mm_Horizontal, F.Cu at (69.1, 37.0)
- added J3: Conn_01x01_Female, Connector_PinHeader_2.54mm:PinHeader_1x01_P2.54mm_Horizontal, F.Cu at (208.9, 173.7)
- added J3: Conn_01x01_Female, Connector_PinHeader_2.54mm:PinHeader_1x01_P2.54mm_Horizontal, F.Cu at (140.9, 173.3)
- added J3: Conn_01x01_Female, Connector_PinHeader_2.54mm:PinHeader_1x01_P2.54mm_Horizontal, F.Cu at (73.5, 173.4)
- added J3: Conn_01x01_Female, Connector_PinHeader_2.54mm:PinHeader_1x01_P2.54mm_Horizontal, F.Cu at (275.1, 132.3)
- added J3: Conn_01x01_Female, Connector_PinHeader_2.54mm:PinHeader_1x01_P2.54mm_Horizontal, F.Cu at (207.7, 132.4)
- added J3: Conn_01x01_Female, Connector_PinHeader_2.54mm:PinHeader_1x01_P2.54mm_Horizontal, F.Cu at (139.7, 132.0)
- added J3: Conn_01x01_Female, Connector_PinHeader_2.54mm:PinHeader_1x01_P2.54mm_Horizontal, F.Cu at (72.4, 132.1)
- added J3: Conn_01x01_Female, Connector_PinHeader_2.54mm:PinHeader_1x01_P2.54mm_Horizontal, F.Cu at (272.8, 86.8)
- added J4: Conn_01x01_Female, Connector_PinHeader_2.54mm:PinHeader_1x01_P2.54mm_Horizontal, F.Cu at (140.6, 183.4)
- added J4: Conn_01x01_Female, Connector_PinHeader_2.54mm:PinHeader_1x01_P2.54mm_Horizontal, F.Cu at (272.5, 97.0)
- added J4: Conn_01x01_Female, Connector_PinHeader_2.54mm:PinHeader_1x01_P2.54mm_Horizontal, F.Cu at (205.2, 97.1)
- added J4: Conn_01x01_Female, Connector_PinHeader_2.54mm:PinHeader_1x01_P2.54mm_Horizontal, F.Cu at (69.8, 96.8)
- added J4: Conn_01x01_Female, Connector_PinHeader_2.54mm:PinHeader_1x01_P2.54mm_Horizontal, F.Cu at (271.5, 47.3)
- added J4: Conn_01x01_Female, Connector_PinHeader_2.54mm:PinHeader_1x01_P2.54mm_Horizontal, F.Cu at (204.2, 47.4)
- added J4: Conn_01x01_Female, Connector_PinHeader_2.54mm:PinHeader_1x01_P2.54mm_Horizontal, F.Cu at (136.2, 47.0)
- added J4: Conn_01x01_Female, Connector_PinHeader_2.54mm:PinHeader_1x01_P2.54mm_Horizontal, F.Cu at (68.9, 47.1)
- added J4: Conn_01x01_Female, Connector_PinHeader_2.54mm:PinHeader_1x01_P2.54mm_Horizontal, F.Cu at (275.9, 183.7)
- added J4: Conn_01x01_Female, Connector_PinHeader_2.54mm:PinHeader_1x01_P2.54mm_Horizontal, F.Cu at (208.6, 183.8)
- added J4: Conn_01x01_Female, Connector_PinHeader_2.54mm:PinHeader_1x01_P2.54mm_Horizontal, F.Cu at (73.3, 183.6)
- added J4: Conn_01x01_Female, Connector_PinHeader_2.54mm:PinHeader_1x01_P2.54mm_Horizontal, F.Cu at (139.5, 142.1)
- added J4: Conn_01x01_Female, Connector_PinHeader_2.54mm:PinHeader_1x01_P2.54mm_Horizontal, F.Cu at (274.8, 142.4)
- added J4: Conn_01x01_Female, Connector_PinHeader_2.54mm:PinHeader_1x01_P2.54mm_Horizontal, F.Cu at (207.5, 142.6)
- added J4: Conn_01x01_Female, Connector_PinHeader_2.54mm:PinHeader_1x01_P2.54mm_Horizontal, F.Cu at (72.1, 142.3)
- added J4: Conn_01x01_Female, Connector_PinHeader_2.54mm:PinHeader_1x01_P2.54mm_Horizontal, F.Cu at (137.2, 96.7)
- added L1: L, Inductor_THT:L_Axial_L16.0mm_D6.3mm_P20.32mm_Horizontal_Fastron_VHBCC, F.Cu at (114.1, 159.9)
- added L1: L, Inductor_THT:L_Axial_L16.0mm_D6.3mm_P20.32mm_Horizontal_Fastron_VHBCC, F.Cu at (246.0, 73.5)
- added L1: L, Inductor_THT:L_Axial_L16.0mm_D6.3mm_P20.32mm_Horizontal_Fastron_VHBCC, F.Cu at (178.6, 73.6)
- added L1: L, Inductor_THT:L_Axial_L16.0mm_D6.3mm_P20.32mm_Horizontal_Fastron_VHBCC, F.Cu at (43.3, 73.3)
- added L1: L, Inductor_THT:L_Axial_L16.0mm_D6.3mm_P20.32mm_Horizontal_Fastron_VHBCC, F.Cu at (245.0, 23.8)
- added L1: L, Inductor_THT:L_Axial_L16.0mm_D6.3mm_P20.32mm_Horizontal_Fastron_VHBCC, F.Cu at (177.6, 23.9)
- added L1: L, Inductor_THT:L_Axial_L16.0mm_D6.3mm_P20.32mm_Horizontal_Fastron_VHBCC, F.Cu at (109.7, 23.5)
- added L1: L, Inductor_THT:L_Axial_L16.0mm_D6.3mm_P20.32mm_Horizontal_Fastron_VHBCC, F.Cu at (42.3, 23.6)
- added L1: L, Inductor_THT:L_Axial_L16.0mm_D6.3mm_P20.32mm_Horizontal_Fastron_VHBCC, F.Cu at (249.4, 160.2)
- added L1: L, Inductor_THT:L_Axial_L16.0mm_D6.3mm_P20.32mm_Horizontal_Fastron_VHBCC, F.Cu at (182.1, 160.4)
- added L1: L, Inductor_THT:L_Axial_L16.0mm_D6.3mm_P20.32mm_Horizontal_Fastron_VHBCC, F.Cu at (46.7, 160.1)
- added L1: L, Inductor_THT:L_Axial_L16.0mm_D6.3mm_P20.32mm_Horizontal_Fastron_VHBCC, F.Cu at (112.9, 118.6)
- added L1: L, Inductor_THT:L_Axial_L16.0mm_D6.3mm_P20.32mm_Horizontal_Fastron_VHBCC, F.Cu at (248.3, 118.9)
- added L1: L, Inductor_THT:L_Axial_L16.0mm_D6.3mm_P20.32mm_Horizontal_Fastron_VHBCC, F.Cu at (180.9, 119.1)
- added L1: L, Inductor_THT:L_Axial_L16.0mm_D6.3mm_P20.32mm_Horizontal_Fastron_VHBCC, F.Cu at (45.6, 118.8)
- added L1: L, Inductor_THT:L_Axial_L16.0mm_D6.3mm_P20.32mm_Horizontal_Fastron_VHBCC, F.Cu at (110.6, 73.2)
- added L2: L, Inductor_THT:L_Axial_L16.0mm_D6.3mm_P20.32mm_Horizontal_Fastron_VHBCC, F.Cu at (118.8, 159.9)
- added L2: L, Inductor_THT:L_Axial_L16.0mm_D6.3mm_P20.32mm_Horizontal_Fastron_VHBCC, F.Cu at (250.7, 73.5)
- added L2: L, Inductor_THT:L_Axial_L16.0mm_D6.3mm_P20.32mm_Horizontal_Fastron_VHBCC, F.Cu at (183.3, 73.6)
- added L2: L, Inductor_THT:L_Axial_L16.0mm_D6.3mm_P20.32mm_Horizontal_Fastron_VHBCC, F.Cu at (48.0, 73.3)
- added L2: L, Inductor_THT:L_Axial_L16.0mm_D6.3mm_P20.32mm_Horizontal_Fastron_VHBCC, F.Cu at (249.7, 23.8)
- added L2: L, Inductor_THT:L_Axial_L16.0mm_D6.3mm_P20.32mm_Horizontal_Fastron_VHBCC, F.Cu at (182.3, 23.9)
- added L2: L, Inductor_THT:L_Axial_L16.0mm_D6.3mm_P20.32mm_Horizontal_Fastron_VHBCC, F.Cu at (114.4, 23.5)
- added L2: L, Inductor_THT:L_Axial_L16.0mm_D6.3mm_P20.32mm_Horizontal_Fastron_VHBCC, F.Cu at (47.0, 23.6)
- added L2: L, Inductor_THT:L_Axial_L16.0mm_D6.3mm_P20.32mm_Horizontal_Fastron_VHBCC, F.Cu at (254.1, 160.2)
- added L2: L, Inductor_THT:L_Axial_L16.0mm_D6.3mm_P20.32mm_Horizontal_Fastron_VHBCC, F.Cu at (186.8, 160.4)
- added L2: L, Inductor_THT:L_Axial_L16.0mm_D6.3mm_P20.32mm_Horizontal_Fastron_VHBCC, F.Cu at (51.4, 160.1)
- added L2: L, Inductor_THT:L_Axial_L16.0mm_D6.3mm_P20.32mm_Horizontal_Fastron_VHBCC, F.Cu at (117.6, 118.6)
- added L2: L, Inductor_THT:L_Axial_L16.0mm_D6.3mm_P20.32mm_Horizontal_Fastron_VHBCC, F.Cu at (253.0, 118.9)
- added L2: L, Inductor_THT:L_Axial_L16.0mm_D6.3mm_P20.32mm_Horizontal_Fastron_VHBCC, F.Cu at (185.6, 119.1)
- added L2: L, Inductor_THT:L_Axial_L16.0mm_D6.3mm_P20.32mm_Horizontal_Fastron_VHBCC, F.Cu at (50.3, 118.8)
- added L2: L, Inductor_THT:L_Axial_L16.0mm_D6.3mm_P20.32mm_Horizontal_Fastron_VHBCC, F.Cu at (115.3, 73.2)
- added Q1: 2N3904, Package_TO_SOT_THT:TO-92L_Inline_Wide, F.Cu at (49.9, 170.7)
- added Q1: 2N3904, Package_TO_SOT_THT:TO-92L_Inline_Wide, F.Cu at (181.8, 84.3)
- added Q1: 2N3904, Package_TO_SOT_THT:TO-92L_Inline_Wide, F.Cu at (249.1, 84.1)
- added Q1: 2N3904, Package_TO_SOT_THT:TO-92L_Inline_Wide, F.Cu at (113.8, 83.8)
- added Q1: 2N3904, Package_TO_SOT_THT:TO-92L_Inline_Wide, F.Cu at (180.8, 34.6)
- added Q1: 2N3904, Package_TO_SOT_THT:TO-92L_Inline_Wide, F.Cu at (248.2, 34.4)
- added Q1: 2N3904, Package_TO_SOT_THT:TO-92L_Inline_Wide, F.Cu at (112.8, 34.2)
- added Q1: 2N3904, Package_TO_SOT_THT:TO-92L_Inline_Wide, F.Cu at (45.5, 34.3)
- added Q1: 2N3904, Package_TO_SOT_THT:TO-92L_Inline_Wide, F.Cu at (185.2, 171.0)
- added Q1: 2N3904, Package_TO_SOT_THT:TO-92L_Inline_Wide, F.Cu at (252.6, 170.9)
- added Q1: 2N3904, Package_TO_SOT_THT:TO-92L_Inline_Wide, F.Cu at (117.2, 170.6)
- added Q1: 2N3904, Package_TO_SOT_THT:TO-92L_Inline_Wide, F.Cu at (48.8, 129.5)
- added Q1: 2N3904, Package_TO_SOT_THT:TO-92L_Inline_Wide, F.Cu at (184.1, 129.7)
- added Q1: 2N3904, Package_TO_SOT_THT:TO-92L_Inline_Wide, F.Cu at (251.4, 129.6)
- added Q1: 2N3904, Package_TO_SOT_THT:TO-92L_Inline_Wide, F.Cu at (116.1, 129.3)
- added Q1: 2N3904, Package_TO_SOT_THT:TO-92L_Inline_Wide, F.Cu at (46.5, 84.0)
- added R1: R, Resistor_THT:R_Axial_DIN0207_L6.3mm_D2.5mm_P10.16mm_Horizontal, F.Cu at (108.2, 171.0)
- added R1: R, Resistor_THT:R_Axial_DIN0207_L6.3mm_D2.5mm_P10.16mm_Horizontal, F.Cu at (240.1, 84.5)
- added R1: R, Resistor_THT:R_Axial_DIN0207_L6.3mm_D2.5mm_P10.16mm_Horizontal, F.Cu at (172.8, 84.7)
- added R1: R, Resistor_THT:R_Axial_DIN0207_L6.3mm_D2.5mm_P10.16mm_Horizontal, F.Cu at (37.5, 84.4)
- added R1: R, Resistor_THT:R_Axial_DIN0207_L6.3mm_D2.5mm_P10.16mm_Horizontal, F.Cu at (239.1, 34.8)
- added R1: R, Resistor_THT:R_Axial_DIN0207_L6.3mm_D2.5mm_P10.16mm_Horizontal, F.Cu at (171.8, 35.0)
- added R1: R, Resistor_THT:R_Axial_DIN0207_L6.3mm_D2.5mm_P10.16mm_Horizontal, F.Cu at (103.8, 34.5)
- added R1: R, Resistor_THT:R_Axial_DIN0207_L6.3mm_D2.5mm_P10.16mm_Horizontal, F.Cu at (36.5, 34.7)
- added R1: R, Resistor_THT:R_Axial_DIN0207_L6.3mm_D2.5mm_P10.16mm_Horizontal, F.Cu at (243.6, 171.2)
- added R1: R, Resistor_THT:R_Axial_DIN0207_L6.3mm_D2.5mm_P10.16mm_Horizontal, F.Cu at (176.2, 171.4)
- added R1: R, Resistor_THT:R_Axial_DIN0207_L6.3mm_D2.5mm_P10.16mm_Horizontal, F.Cu at (40.9, 171.1)
- added R1: R, Resistor_THT:R_Axial_DIN0207_L6.3mm_D2.5mm_P10.16mm_Horizontal, F.Cu at (107.1, 129.7)
- added R1: R, Resistor_THT:R_Axial_DIN0207_L6.3mm_D2.5mm_P10.16mm_Horizontal, F.Cu at (242.4, 130.0)
- added R1: R, Resistor_THT:R_Axial_DIN0207_L6.3mm_D2.5mm_P10.16mm_Horizontal, F.Cu at (175.1, 130.1)
- added R1: R, Resistor_THT:R_Axial_DIN0207_L6.3mm_D2.5mm_P10.16mm_Horizontal, F.Cu at (39.8, 129.8)
- added R1: R, Resistor_THT:R_Axial_DIN0207_L6.3mm_D2.5mm_P10.16mm_Horizontal, F.Cu at (104.8, 84.2)
- added R2: R, Resistor_THT:R_Axial_DIN0207_L6.3mm_D2.5mm_P10.16mm_Horizontal, F.Cu at (98.1, 166.4)
- added R2: R, Resistor_THT:R_Axial_DIN0207_L6.3mm_D2.5mm_P10.16mm_Horizontal, F.Cu at (230.0, 79.9)
- added R2: R, Resistor_THT:R_Axial_DIN0207_L6.3mm_D2.5mm_P10.16mm_Horizontal, F.Cu at (162.6, 80.1)
- added R2: R, Resistor_THT:R_Axial_DIN0207_L6.3mm_D2.5mm_P10.16mm_Horizontal, F.Cu at (27.3, 79.8)
- added R2: R, Resistor_THT:R_Axial_DIN0207_L6.3mm_D2.5mm_P10.16mm_Horizontal, F.Cu at (229.0, 30.3)
- added R2: R, Resistor_THT:R_Axial_DIN0207_L6.3mm_D2.5mm_P10.16mm_Horizontal, F.Cu at (161.6, 30.4)
- added R2: R, Resistor_THT:R_Axial_DIN0207_L6.3mm_D2.5mm_P10.16mm_Horizontal, F.Cu at (93.6, 30.0)
- added R2: R, Resistor_THT:R_Axial_DIN0207_L6.3mm_D2.5mm_P10.16mm_Horizontal, F.Cu at (26.3, 30.1)
- added R2: R, Resistor_THT:R_Axial_DIN0207_L6.3mm_D2.5mm_P10.16mm_Horizontal, F.Cu at (233.4, 166.7)
- added R2: R, Resistor_THT:R_Axial_DIN0207_L6.3mm_D2.5mm_P10.16mm_Horizontal, F.Cu at (166.1, 166.8)
- added R2: R, Resistor_THT:R_Axial_DIN0207_L6.3mm_D2.5mm_P10.16mm_Horizontal, F.Cu at (30.7, 166.5)
- added R2: R, Resistor_THT:R_Axial_DIN0207_L6.3mm_D2.5mm_P10.16mm_Horizontal, F.Cu at (96.9, 125.1)
- added R2: R, Resistor_THT:R_Axial_DIN0207_L6.3mm_D2.5mm_P10.16mm_Horizontal, F.Cu at (232.3, 125.4)
- added R2: R, Resistor_THT:R_Axial_DIN0207_L6.3mm_D2.5mm_P10.16mm_Horizontal, F.Cu at (164.9, 125.6)
- added R2: R, Resistor_THT:R_Axial_DIN0207_L6.3mm_D2.5mm_P10.16mm_Horizontal, F.Cu at (29.6, 125.3)
- added R2: R, Resistor_THT:R_Axial_DIN0207_L6.3mm_D2.5mm_P10.16mm_Horizontal, F.Cu at (94.6, 79.7)
- added R3: R, Resistor_THT:R_Axial_DIN0207_L6.3mm_D2.5mm_P10.16mm_Horizontal, F.Cu at (135.2, 173.3)
- added R3: R, Resistor_THT:R_Axial_DIN0207_L6.3mm_D2.5mm_P10.16mm_Horizontal, F.Cu at (267.1, 86.8)
- added R3: R, Resistor_THT:R_Axial_DIN0207_L6.3mm_D2.5mm_P10.16mm_Horizontal, F.Cu at (199.7, 86.9)
- added R3: R, Resistor_THT:R_Axial_DIN0207_L6.3mm_D2.5mm_P10.16mm_Horizontal, F.Cu at (64.4, 86.7)
- added R3: R, Resistor_THT:R_Axial_DIN0207_L6.3mm_D2.5mm_P10.16mm_Horizontal, F.Cu at (266.1, 37.1)
- added R3: R, Resistor_THT:R_Axial_DIN0207_L6.3mm_D2.5mm_P10.16mm_Horizontal, F.Cu at (198.7, 37.3)
- added R3: R, Resistor_THT:R_Axial_DIN0207_L6.3mm_D2.5mm_P10.16mm_Horizontal, F.Cu at (130.7, 36.8)
- added R3: R, Resistor_THT:R_Axial_DIN0207_L6.3mm_D2.5mm_P10.16mm_Horizontal, F.Cu at (63.4, 37.0)
- added R3: R, Resistor_THT:R_Axial_DIN0207_L6.3mm_D2.5mm_P10.16mm_Horizontal, F.Cu at (270.5, 173.5)
- added R3: R, Resistor_THT:R_Axial_DIN0207_L6.3mm_D2.5mm_P10.16mm_Horizontal, F.Cu at (203.1, 173.7)
- added R3: R, Resistor_THT:R_Axial_DIN0207_L6.3mm_D2.5mm_P10.16mm_Horizontal, F.Cu at (67.8, 173.4)
- added R3: R, Resistor_THT:R_Axial_DIN0207_L6.3mm_D2.5mm_P10.16mm_Horizontal, F.Cu at (134.0, 132.0)
- added R3: R, Resistor_THT:R_Axial_DIN0207_L6.3mm_D2.5mm_P10.16mm_Horizontal, F.Cu at (269.3, 132.3)
- added R3: R, Resistor_THT:R_Axial_DIN0207_L6.3mm_D2.5mm_P10.16mm_Horizontal, F.Cu at (202.0, 132.4)
- added R3: R, Resistor_THT:R_Axial_DIN0207_L6.3mm_D2.5mm_P10.16mm_Horizontal, F.Cu at (66.7, 132.1)
- added R3: R, Resistor_THT:R_Axial_DIN0207_L6.3mm_D2.5mm_P10.16mm_Horizontal, F.Cu at (131.7, 86.5)
- added RV1: R_POT, Potentiometer_THT:Potentiometer_Alps_RK163_Single_Horizontal, F.Cu at (100.1, 180.4)
- added RV1: R_POT, Potentiometer_THT:Potentiometer_Alps_RK163_Single_Horizontal, F.Cu at (232.0, 93.9)
- added RV1: R_POT, Potentiometer_THT:Potentiometer_Alps_RK163_Single_Horizontal, F.Cu at (164.6, 94.1)
- added RV1: R_POT, Potentiometer_THT:Potentiometer_Alps_RK163_Single_Horizontal, F.Cu at (29.3, 93.8)
- added RV1: R_POT, Potentiometer_THT:Potentiometer_Alps_RK163_Single_Horizontal, F.Cu at (231.0, 44.2)
- added RV1: R_POT, Potentiometer_THT:Potentiometer_Alps_RK163_Single_Horizontal, F.Cu at (163.6, 44.4)
- added RV1: R_POT, Potentiometer_THT:Potentiometer_Alps_RK163_Single_Horizontal, F.Cu at (95.6, 43.9)
- added RV1: R_POT, Potentiometer_THT:Potentiometer_Alps_RK163_Single_Horizontal, F.Cu at (28.3, 44.1)
- added RV1: R_POT, Potentiometer_THT:Potentiometer_Alps_RK163_Single_Horizontal, F.Cu at (235.4, 180.6)
- added RV1: R_POT, Potentiometer_THT:Potentiometer_Alps_RK163_Single_Horizontal, F.Cu at (168.1, 180.8)
- added RV1: R_POT, Potentiometer_THT:Potentiometer_Alps_RK163_Single_Horizontal, F.Cu at (32.7, 180.5)
- added RV1: R_POT, Potentiometer_THT:Potentiometer_Alps_RK163_Single_Horizontal, F.Cu at (98.9, 139.1)
- added RV1: R_POT, Potentiometer_THT:Potentiometer_Alps_RK163_Single_Horizontal, F.Cu at (234.2, 139.4)
- added RV1: R_POT, Potentiometer_THT:Potentiometer_Alps_RK163_Single_Horizontal, F.Cu at (166.9, 139.5)
- added RV1: R_POT, Potentiometer_THT:Potentiometer_Alps_RK163_Single_Horizontal, F.Cu at (31.6, 139.2)
- added RV1: R_POT, Potentiometer_THT:Potentiometer_Alps_RK163_Single_Horizontal, F.Cu at (96.6, 93.6)
- added RV2: R_POT, Potentiometer_THT:Potentiometer_Alps_RK163_Single_Horizontal, F.Cu at (119.3, 180.4)
- added RV2: R_POT, Potentiometer_THT:Potentiometer_Alps_RK163_Single_Horizontal, F.Cu at (251.2, 93.9)
- added RV2: R_POT, Potentiometer_THT:Potentiometer_Alps_RK163_Single_Horizontal, F.Cu at (183.8, 94.1)
- added RV2: R_POT, Potentiometer_THT:Potentiometer_Alps_RK163_Single_Horizontal, F.Cu at (48.5, 93.8)
- added RV2: R_POT, Potentiometer_THT:Potentiometer_Alps_RK163_Single_Horizontal, F.Cu at (250.2, 44.2)
- added RV2: R_POT, Potentiometer_THT:Potentiometer_Alps_RK163_Single_Horizontal, F.Cu at (182.9, 44.4)
- added RV2: R_POT, Potentiometer_THT:Potentiometer_Alps_RK163_Single_Horizontal, F.Cu at (114.9, 43.9)
- added RV2: R_POT, Potentiometer_THT:Potentiometer_Alps_RK163_Single_Horizontal, F.Cu at (47.5, 44.1)
- added RV2: R_POT, Potentiometer_THT:Potentiometer_Alps_RK163_Single_Horizontal, F.Cu at (254.6, 180.6)
- added RV2: R_POT, Potentiometer_THT:Potentiometer_Alps_RK163_Single_Horizontal, F.Cu at (187.3, 180.8)
- added RV2: R_POT, Potentiometer_THT:Potentiometer_Alps_RK163_Single_Horizontal, F.Cu at (51.9, 180.5)
- added RV2: R_POT, Potentiometer_THT:Potentiometer_Alps_RK163_Single_Horizontal, F.Cu at (118.1, 139.1)
- added RV2: R_POT, Potentiometer_THT:Potentiometer_Alps_RK163_Single_Horizontal, F.Cu at (253.5, 139.4)
- added RV2: R_POT, Potentiometer_THT:Potentiometer_Alps_RK163_Single_Horizontal, F.Cu at (186.1, 139.5)
- added RV2: R_POT, Potentiometer_THT:Potentiometer_Alps_RK163_Single_Horizontal, F.Cu at (50.8, 139.2)
- added RV2: R_POT, Potentiometer_THT:Potentiometer_Alps_RK163_Single_Horizontal, F.Cu at (115.8, 93.6)
Routing:
- net (no net): track 1043.7 -> 4705.8 mm, vias 4 -> 0
- net Net-(C1-Pad2): track 92.5 -> 0.00 mm
- net Net-(C3-Pad2): track 66.7 -> 10.2 mm
- net Net-(C1-Pad1): track 63.8 -> 14.0 mm, vias 1 -> 0
- net Net-(J1-Pad1): track 42.6 -> 0.00 mm
- net Net-(C2-Pad2): track 0.00 -> 42.4 mm
- net Net-(C3-Pad1): track 91.9 -> 49.8 mm, vias 1 -> 0
- net +12V: track 0.00 -> 15.1 mm
- net Net-(C4-Pad1): track 0.00 -> 9.95 mm
- net GND: track 136.3 -> 143.6 mm
- net Net-(C2-Pad1): track 28.0 -> 28.6 mm
- added copper zone on F.Cu, net GND
Other:
- board outline added: 262.1 x 168.6 mm
