File: Electronica de Potencia/TP's/TPN3/PCB/PWM/SG3525A/SG3525A.kicad_pcb (KiCad board)
At the start: 2 copper layers, 40.3 x 37.5 mm, 17 parts, among them J1 Vin, J2 PWM_out, U1 SG3525

Commit message: Actualizo repo
Parts:
- moved C2 0.63 mm to (151.1, 103.4)
Routing:
- net Net-(C2-Pad1): track 12.7 -> 13.8 mm
Other:
- board text added: "+15V"
Changed lines of the file:
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@@
   (general
     (thickness 1.6)
-    (drawings 11)
+    (drawings 13)
     (tracks 85)
     (zones 0)
@@
     (mod_text_size 1 1)
     (mod_text_width 0.15)
-    (pad_size 3 3)
-    (pad_drill 1.52)
+    (pad_size 2 2)
+    (pad_drill 0.8)
     (pad_to_mask_clearance 0.051)
     (solder_mask_min_width 0.25)
@@
       (effects (font (size 0.94 0.94) (thickness 0.141)))
     )
-    (pad 1 thru_hole circle (at 0 0 270) (size 1.6 1.6) (drill 0.8) (layers *.Cu *.Mask)
+    (pad 1 thru_hole circle (at 0 0 270) (size 2 2) (drill 0.8) (layers *.Cu *.Mask)
       (net 1 "Net-(C1-Pad1)"))
-    (pad 2 thru_hole circle (at 5 0 270) (size 1.6 1.6) (drill 0.8) (layers *.Cu *.Mask)
+    (pad 2 thru_hole circle (at 5 0 270) (size 2 2) (drill 0.8) (layers *.Cu *.Mask)
       (net 2 Earth))
     (model ${KISYS3DMOD}/Capacitor_THT.3dshapes/C_Disc_D4.7mm_W2.5mm_P5.00mm.wrl
@@
   )
   (module lib_fp:C_Radial_D5.0mm_H11.0mm_P2.00mm (layer F.Cu)
-    (at 150.495 103.4415 270)
+    (at 151.13 103.4415 270)
     (descr "C, Radial series, Radial, pin pitch=2.00mm, diameter=5mm, height=11mm, Non-Polar Electrolytic Capacitor")
     (tags "C Radial series Radial pin pitch 2.00mm diameter 5mm height 11mm Non-Polar Electrolytic Capacitor")
@@
     (descr "simple 2-pin terminal block, pitch 5.08mm, revamped version of bornier2")
     (tags "terminal block bornier2")
-    (fp_text reference J1 (at 2.54 -5.08 90) (layer F.SilkS)
+    (fp_text reference J1 (at -0.004 -5.0854 90) (layer F.SilkS)
       (effects (font (size 1 1) (thickness 0.15)))
     )
@@
       (effects (font (size 1 1) (thickness 0.15)))
     )
-    (pad 2 thru_hole circle (at 5.08 0 90) (size 3 3) (drill 1.52) (layers *.Cu *.Mask)
+    (pad 2 thru_hole circle (at 5.08 0 90) (size 3 3) (drill 1.2) (layers *.Cu *.Mask)
       (net 5 +12V))
-    (pad 1 thru_hole rect (at 0 0 90) (size 3 3) (drill 1.52) (layers *.Cu *.Mask)
+    (pad 1 thru_hole circle (at 0 0 90) (size 3 3) (drill 1.2) (layers *.Cu *.Mask)
       (net 2 Earth))
     (model "${KIPRJMOD}/3d_models/User Library-Terminal block 2 POS/User Library-Terminal block 2 POS.STEP"
@@
     (descr "Potentiometer, vertical, Bourns 3266Y, https://www.bourns.com/docs/Product-Datasheets/3266.pdf")
     (tags "Potentiometer vertical Bourns 3266Y")
-    (fp_text reference RV2 (at -1.27 3.556 180) (layer F.SilkS)
+    (fp_text reference RV2 (at -2.6162 3.3528 180) (layer F.SilkS)
       (effects (font (size 1 1) (thickness 0.15)))
     )
@@
     (descr "16-lead though-hole mounted DIP package, row spacing 7.62 mm (300 mils), LongPads")
     (tags "THT DIP DIL PDIP 2.54mm 7.62mm 300mil LongPads")
-    (fp_text reference U1 (at 4.064 20.35) (layer F.SilkS)
+    (fp_text reference U1 (at 3.8735 20.0025) (layer F.SilkS)
       (effects (font (size 1 1) (thickness 0.15)))
     )
@@
     (fp_line (start 12.88 4) (end 12.88 -4) (layer F.CrtYd) (width 0.05))
     (fp_line (start 12.88 4) (end -2.72 4) (layer F.CrtYd) (width 0.05))
-    (pad 1 thru_hole rect (at 0 0 90) (size 3 3) (drill 1.52) (layers *.Cu *.Mask)
+    (pad 1 thru_hole rect (at 0 0 90) (size 3 3) (drill 1.2) (layers *.Cu *.Mask)
       (net 7 /PWM_A))
-    (pad 2 thru_hole circle (at 5.08 0 90) (size 3 3) (drill 1.52) (layers *.Cu *.Mask)
-      (net 2 Earth))
-    (pad 3 thru_hole circle (at 10.16 0 90) (size 3 3) (drill 1.52) (layers *.Cu *.Mask)
+    (pad 2 thru_hole circle (at 5.08 0 90) (size 3 3) (drill 1.2) (layers *.Cu *.Mask)
+      (net 2 Earth))
+    (pad 3 thru_hole circle (at 10.16 0 90) (size 3 3) (drill 1.2) (layers *.Cu *.Mask)
       (net 6 /PWM_B))
     (model "${KIPRJMOD}/3d_models/User Library-Terminal block 3 POS/User Library-Terminal block 3 POS.STEP"
@@
     )
   )
-  (gr_text "Duty Cicle" (at 136.144 105.41) (layer F.SilkS)
+  (gr_text - (at 132.969 105.9942 90) (layer F.SilkS)
+    (effects (font (size 2 2) (thickness 0.15)))
+  )
+  (gr_text +15V (at 122.8852 100.838 90) (layer F.SilkS)
+    (effects (font (size 1 1) (thickness 0.15)))
+  )
+  (gr_text "Duty Cicle" (at 144.0688 108.5596) (layer F.SilkS)
     (effects (font (size 1 1) (thickness 0.15)))
   )
@@
     (effects (font (size 1 1) (thickness 0.15)))
   )
-  (gr_text + (at 132.996 100.514) (layer F.SilkS)
-    (effects (font (size 1 1) (thickness 0.15)))
+  (gr_text + (at 133.1468 100.7364) (layer F.SilkS)
+    (effects (font (size 2 2) (thickness 0.15)))
   )
   (gr_line (start 162.096 72.014) (end 161.596 72.014) (layer Edge.Cuts) (width 0.05))
@@
   (segment (start 140.97 90.424) (end 138.43 92.964) (width 0.8) (layer B.Cu) (net 1) (status 10))
   (segment (start 137.16 92.964) (end 133.604 92.964) (width 0.8) (layer B.Cu) (net 1) (status 30))
-  (segment (start 141.732 100.965) (end 141.732 98.044) (width 0.8) (layer B.Cu) (net 3) (status 20))
-  (segment (start 150.495 103.4415) (end 144.2085 103.4415) (width 0.8) (layer B.Cu) (net 3) (status 10))
-  (segment (start 144.2085 103.4415) (end 141.732 100.965) (width 0.8) (layer B.Cu) (net 3))
+  (segment (start 151.13 103.4415) (end 143.4465 103.4415) (width 0.8) (layer B.Cu) (net 3))
+  (segment (start 141.732 101.727) (end 141.732 98.044) (width 0.8) (layer B.Cu) (net 3))
+  (segment (start 143.4465 103.4415) (end 141.732 101.727) (width 0.8) (layer B.Cu) (net 3))
   (segment (start 126.596 92.414) (end 127.696 93.514) (width 0.8) (layer B.Cu) (net 4) (status 20))
   (segment (start 126.596 90.374) (end 126.596 92.414) (width 0.8) (layer B.Cu) (net 4) (status 10))
