File: Electronica de Potencia/TP's/TPN3/PCB/PWM/SG3525A/SG3525A_PANEL.kicad_pcb (KiCad board)
At the start: 2 copper layers, 231.5 x 153.5 mm, 204 parts, among them J1 Vin, J2 PWM_out, U1 SG3525

Commit message: Actualizo repo
Parts:
- removed the C1 at (56.4, 158.3)
- removed the C1 at (241.8, 42.3)
- removed the C1 at (117.6, 43.7)
- removed the C1 at (54.3, 43.8)
- removed the C1 at (180.6, 156.9)
- removed the C1 at (244.0, 156.9)
- removed the C1 at (119.8, 158.3)
- removed the C1 at (52.8, 99.5)
- removed the C1 at (176.9, 98.1)
- removed the C1 at (240.3, 98.1)
- removed the C1 at (116.2, 99.5)
- removed the C1 at (178.4, 42.4)
- removed the C2 at (73.3, 168.8)
- removed the C2 at (258.7, 52.8)
- removed the C2 at (134.5, 54.2)
- removed the C2 at (71.1, 54.3)
- removed the C2 at (260.9, 167.3)
- removed the C2 at (136.7, 168.7)
- removed the C2 at (197.5, 167.4)
- removed the C2 at (69.6, 110.0)
- removed the C2 at (257.2, 108.6)
- removed the C2 at (133.0, 110.0)
- removed the C2 at (193.8, 108.6)
- removed the C2 at (195.3, 52.9)
- removed the D1 at (50.5, 158.9)
- removed the D1 at (235.9, 42.9)
- removed the D1 at (111.7, 44.3)
- removed the D1 at (48.3, 44.3)
- removed the D1 at (238.1, 157.4)
- removed the D1 at (113.9, 158.8)
- removed the D1 at (174.7, 157.5)
- removed the D1 at (46.8, 100.1)
- removed the D1 at (234.4, 98.6)
- removed the D1 at (110.2, 100.0)
- removed the D1 at (171.0, 98.7)
- removed the D1 at (172.5, 42.9)
- removed the G1 at (49.4, 141.1)
- removed the G1 at (234.8, 25.1)
- removed the G1 at (110.6, 26.5)
- removed the G1 at (47.2, 26.5)
- removed the G1 at (173.6, 139.7)
- removed the G1 at (237.0, 139.6)
- removed the G1 at (112.8, 141.0)
- removed the G1 at (45.7, 82.3)
- removed the G1 at (169.9, 80.9)
- removed the G1 at (233.3, 80.8)
- removed the G1 at (109.1, 82.2)
- removed the G1 at (171.4, 25.1)
- removed the J1 at (50.8, 171.3)
- removed the J1 at (236.2, 55.3)
- removed the J1 at (112.0, 56.7)
- removed the J1 at (48.6, 56.7)
- removed the J1 at (175.0, 169.9)
- removed the J1 at (114.2, 171.2)
- removed the J1 at (238.4, 169.8)
- removed the J1 at (47.1, 112.5)
- removed the J1 at (171.3, 111.1)
- removed the J1 at (110.5, 112.4)
- removed the J1 at (234.7, 111.0)
- removed the J1 at (172.8, 55.3)
- removed the J2 at (143.4, 157.4)
- removed the J2 at (202.0, 41.5)
- removed the J2 at (141.2, 42.9)
- removed the J2 at (77.8, 42.9)
- removed the J2 at (80.0, 157.4)
- removed the J2 at (267.6, 156.0)
- removed the J2 at (204.2, 156.0)
- removed the J2 at (139.7, 98.6)
- removed the J2 at (76.3, 98.7)
- removed the J2 at (263.9, 97.2)
- removed the J2 at (200.5, 97.3)
- removed the J2 at (265.4, 41.5)
- removed the R1 at (53.0, 155.9)
- removed the R1 at (238.4, 39.9)
- removed the R1 at (114.2, 41.3)
- removed the R1 at (50.8, 41.3)
- removed the R1 at (116.4, 155.8)
- removed the R1 at (240.6, 154.4)
- removed the R1 at (177.2, 154.5)
- removed the R1 at (49.3, 97.1)
- removed the R1 at (112.7, 97.0)
- removed the R1 at (236.9, 95.6)
- removed the R1 at (173.5, 95.7)
- removed the R1 at (175.0, 39.9)
- removed the R2 at (119.9, 145.6)
- removed the R2 at (178.5, 29.7)
- removed the R2 at (117.7, 31.1)
- removed the R2 at (54.3, 31.1)
- removed the R2 at (244.1, 144.2)
- removed the R2 at (56.5, 145.7)
- removed the R2 at (180.7, 144.3)
- removed the R2 at (116.2, 86.8)
- removed the R2 at (240.4, 85.4)
- removed the R2 at (52.8, 86.9)
- removed the R2 at (177.0, 85.5)
- removed the R2 at (241.9, 29.7)
- removed the R3 at (137.1, 142.0)
- removed the R3 at (195.7, 26.1)
- removed the R3 at (134.9, 27.5)
- removed the R3 at (71.5, 27.5)
- removed the R3 at (261.3, 140.6)
- removed the R3 at (197.9, 140.7)
- removed the R3 at (73.7, 142.1)
- removed the R3 at (133.4, 83.2)
- removed the R3 at (257.6, 81.8)
- removed the R3 at (194.2, 81.9)
- removed the R3 at (70.0, 83.3)
- removed the R3 at (259.1, 26.1)
- removed the R4 at (60.0, 155.8)
- removed the R4 at (245.4, 39.8)
- removed the R4 at (121.2, 41.2)
- removed the R4 at (57.8, 41.2)
- removed the R4 at (123.4, 155.7)
- removed the R4 at (247.5, 154.3)
- removed the R4 at (184.1, 154.4)
- removed the R4 at (56.3, 97.0)
- removed the R4 at (119.7, 96.9)
- removed the R4 at (243.9, 95.5)
- removed the R4 at (180.5, 95.6)
- removed the R4 at (182.0, 39.8)
- removed the R5 at (123.4, 158.3)
- removed the R5 at (182.0, 42.4)
- removed the R5 at (121.2, 43.7)
- removed the R5 at (57.8, 43.8)
- removed the R5 at (184.1, 156.9)
- removed the R5 at (60.0, 158.3)
- removed the R5 at (247.5, 156.9)
- removed the R5 at (119.7, 99.5)
- removed the R5 at (180.5, 98.1)
- removed the R5 at (56.3, 99.5)
- removed the R5 at (243.9, 98.1)
- removed the R5 at (245.4, 42.3)
- removed the R6 at (145.7, 172.0)
- removed the R6 at (204.3, 56.2)
- removed the R6 at (143.5, 57.5)
- removed the R6 at (80.1, 57.6)
- removed the R6 at (269.9, 170.6)
- removed the R6 at (206.5, 170.7)
- removed the R6 at (82.3, 172.1)
- removed the R6 at (142.0, 113.3)
- removed the R6 at (266.2, 111.9)
- removed the R6 at (202.8, 111.9)
- removed the R6 at (78.6, 113.3)
- removed the R6 at (267.7, 56.1)
- removed the R7 at (141.8, 172.0)
- removed the R7 at (200.4, 56.1)
- removed the R7 at (139.6, 57.4)
- removed the R7 at (76.2, 57.5)
- removed the R7 at (78.4, 172.0)
- removed the R7 at (202.6, 170.6)
- removed the R7 at (266.0, 170.6)
- removed the R7 at (138.1, 113.2)
- removed the R7 at (74.7, 113.3)
- removed the R7 at (198.9, 111.9)
- removed the R7 at (262.3, 111.8)
- removed the R7 at (263.8, 56.1)
- removed the R8 at (112.8, 155.7)
- removed the R8 at (171.4, 39.8)
- removed the R8 at (110.6, 41.1)
- removed the R8 at (47.2, 41.2)
- removed the R8 at (49.4, 155.7)
- removed the R8 at (173.6, 154.3)
- removed the R8 at (237.0, 154.3)
- removed the R8 at (109.1, 96.9)
- removed the R8 at (45.7, 96.9)
- removed the R8 at (169.9, 95.6)
- removed the R8 at (233.3, 95.5)
- removed the R8 at (234.8, 39.7)
- removed the RV1 at (77.6, 141.4)
- removed the RV1 at (263.1, 25.4)
- removed the RV1 at (138.9, 26.8)
- removed the RV1 at (75.5, 26.8)
- removed the RV1 at (141.0, 141.3)
- removed the RV1 at (201.8, 140.0)
- removed the RV1 at (265.2, 139.9)
- removed the RV1 at (74.0, 82.6)
- removed the RV1 at (137.4, 82.5)
- removed the RV1 at (198.2, 81.2)
- removed the RV1 at (261.6, 81.1)
- removed the RV1 at (199.7, 25.4)
- removed the RV2 at (127.7, 170.7)
- removed the RV2 at (186.3, 54.8)
- removed the RV2 at (125.5, 56.2)
- removed the RV2 at (62.1, 56.2)
- removed the RV2 at (188.5, 169.4)
- removed the RV2 at (64.3, 170.8)
- removed the RV2 at (251.9, 169.3)
- removed the RV2 at (124.0, 111.9)
- removed the RV2 at (184.8, 110.6)
- removed the RV2 at (60.6, 112.0)
- removed the RV2 at (248.2, 110.5)
- removed the RV2 at (249.7, 54.8)
- removed the U1 at (127.9, 145.6)
- removed the U1 at (186.6, 29.7)
- removed the U1 at (125.8, 31.0)
- removed the U1 at (62.4, 31.1)
- removed the U1 at (188.7, 144.2)
- removed the U1 at (64.5, 145.6)
- removed the U1 at (252.1, 144.2)
- removed the U1 at (124.3, 86.8)
- removed the U1 at (185.1, 85.4)
- removed the U1 at (60.9, 86.8)
- removed the U1 at (248.5, 85.4)
- removed the U1 at (250.0, 29.6)
- added C1: 1nF, lib_fp:C_Disc_D4.7mm_W2.5mm_P5.00mm, F.Cu at (169.8, 163.7)
- added C1: 1nF, lib_fp:C_Disc_D4.7mm_W2.5mm_P5.00mm, F.Cu at (238.7, 46.2)
- added C1: 1nF, lib_fp:C_Disc_D4.7mm_W2.5mm_P5.00mm, F.Cu at (170.4, 46.2)
- added C1: 1nF, lib_fp:C_Disc_D4.7mm_W2.5mm_P5.00mm, F.Cu at (37.2, 46.4)
- added C1: 1nF, lib_fp:C_Disc_D4.7mm_W2.5mm_P5.00mm, F.Cu at (238.0, 163.7)
- added C1: 1nF, lib_fp:C_Disc_D4.7mm_W2.5mm_P5.00mm, F.Cu at (102.8, 163.7)
- added C1: 1nF, lib_fp:C_Disc_D4.7mm_W2.5mm_P5.00mm, F.Cu at (36.5, 163.9)
- added C1: 1nF, lib_fp:C_Disc_D4.7mm_W2.5mm_P5.00mm, F.Cu at (171.7, 104.7)
- added C1: 1nF, lib_fp:C_Disc_D4.7mm_W2.5mm_P5.00mm, F.Cu at (239.9, 104.7)
- added C1: 1nF, lib_fp:C_Disc_D4.7mm_W2.5mm_P5.00mm, F.Cu at (104.7, 104.7)
- added C1: 1nF, lib_fp:C_Disc_D4.7mm_W2.5mm_P5.00mm, F.Cu at (38.4, 104.9)
- added C1: 1nF, lib_fp:C_Disc_D4.7mm_W2.5mm_P5.00mm, F.Cu at (103.5, 46.2)
- added C2: 10uF, lib_fp:C_Radial_D5.0mm_H11.0mm_P2.00mm, F.Cu at (187.3, 174.2)
- added C2: 10uF, lib_fp:C_Radial_D5.0mm_H11.0mm_P2.00mm, F.Cu at (256.2, 56.7)
- added C2: 10uF, lib_fp:C_Radial_D5.0mm_H11.0mm_P2.00mm, F.Cu at (188.0, 56.7)
- added C2: 10uF, lib_fp:C_Radial_D5.0mm_H11.0mm_P2.00mm, F.Cu at (54.7, 56.9)
- added C2: 10uF, lib_fp:C_Radial_D5.0mm_H11.0mm_P2.00mm, F.Cu at (120.4, 174.2)
- added C2: 10uF, lib_fp:C_Radial_D5.0mm_H11.0mm_P2.00mm, F.Cu at (255.6, 174.2)
- added C2: 10uF, lib_fp:C_Radial_D5.0mm_H11.0mm_P2.00mm, F.Cu at (54.1, 174.4)
- added C2: 10uF, lib_fp:C_Radial_D5.0mm_H11.0mm_P2.00mm, F.Cu at (189.2, 115.2)
- added C2: 10uF, lib_fp:C_Radial_D5.0mm_H11.0mm_P2.00mm, F.Cu at (122.2, 115.1)
- added C2: 10uF, lib_fp:C_Radial_D5.0mm_H11.0mm_P2.00mm, F.Cu at (257.5, 115.2)
- added C2: 10uF, lib_fp:C_Radial_D5.0mm_H11.0mm_P2.00mm, F.Cu at (56.0, 115.4)
- added C2: 10uF, lib_fp:C_Radial_D5.0mm_H11.0mm_P2.00mm, F.Cu at (121.0, 56.6)
- added D1: LED, lib_fp:LED_D3.0mm_Clear, F.Cu at (163.9, 164.3)
- added D1: LED, lib_fp:LED_D3.0mm_Clear, F.Cu at (232.8, 46.8)
- added D1: LED, lib_fp:LED_D3.0mm_Clear, F.Cu at (164.5, 46.8)
- added D1: LED, lib_fp:LED_D3.0mm_Clear, F.Cu at (31.3, 47.0)
- added D1: LED, lib_fp:LED_D3.0mm_Clear, F.Cu at (96.9, 164.2)
- added D1: LED, lib_fp:LED_D3.0mm_Clear, F.Cu at (232.1, 164.3)
- added D1: LED, lib_fp:LED_D3.0mm_Clear, F.Cu at (30.6, 164.5)
- added D1: LED, lib_fp:LED_D3.0mm_Clear, F.Cu at (165.7, 105.3)
- added D1: LED, lib_fp:LED_D3.0mm_Clear, F.Cu at (98.8, 105.2)
- added D1: LED, lib_fp:LED_D3.0mm_Clear, F.Cu at (234.0, 105.3)
- added D1: LED, lib_fp:LED_D3.0mm_Clear, F.Cu at (32.5, 105.4)
- added D1: LED, lib_fp:LED_D3.0mm_Clear, F.Cu at (97.6, 46.7)
- added G1: logo, lib_fp:logo_utn_fsilk_small, F.Cu at (162.8, 146.5)
- added G1: logo, lib_fp:logo_utn_fsilk_small, F.Cu at (231.7, 29.0)
- added G1: logo, lib_fp:logo_utn_fsilk_small, F.Cu at (163.4, 29.0)
- added G1: logo, lib_fp:logo_utn_fsilk_small, F.Cu at (30.2, 29.2)
- added G1: logo, lib_fp:logo_utn_fsilk_small, F.Cu at (231.0, 146.5)
- added G1: logo, lib_fp:logo_utn_fsilk_small, F.Cu at (95.8, 146.4)
- added G1: logo, lib_fp:logo_utn_fsilk_small, F.Cu at (29.5, 146.7)
- added G1: logo, lib_fp:logo_utn_fsilk_small, F.Cu at (164.6, 87.5)
- added G1: logo, lib_fp:logo_utn_fsilk_small, F.Cu at (232.9, 87.5)
- added G1: logo, lib_fp:logo_utn_fsilk_small, F.Cu at (97.7, 87.4)
- added G1: logo, lib_fp:logo_utn_fsilk_small, F.Cu at (31.4, 87.6)
- added G1: logo, lib_fp:logo_utn_fsilk_small, F.Cu at (96.5, 28.9)
- added J1: Vin, lib_fp:TerminalBlock_bornier-2_P5.08mm, F.Cu at (164.2, 176.7)
- added J1: Vin, lib_fp:TerminalBlock_bornier-2_P5.08mm, F.Cu at (233.1, 59.2)
- added J1: Vin, lib_fp:TerminalBlock_bornier-2_P5.08mm, F.Cu at (164.8, 59.2)
- added J1: Vin, lib_fp:TerminalBlock_bornier-2_P5.08mm, F.Cu at (31.6, 59.4)
- added J1: Vin, lib_fp:TerminalBlock_bornier-2_P5.08mm, F.Cu at (232.4, 176.7)
- added J1: Vin, lib_fp:TerminalBlock_bornier-2_P5.08mm, F.Cu at (97.2, 176.6)
- added J1: Vin, lib_fp:TerminalBlock_bornier-2_P5.08mm, F.Cu at (30.9, 176.9)
- added J1: Vin, lib_fp:TerminalBlock_bornier-2_P5.08mm, F.Cu at (166.0, 117.7)
- added J1: Vin, lib_fp:TerminalBlock_bornier-2_P5.08mm, F.Cu at (234.3, 117.7)
- added J1: Vin, lib_fp:TerminalBlock_bornier-2_P5.08mm, F.Cu at (99.1, 117.6)
- added J1: Vin, lib_fp:TerminalBlock_bornier-2_P5.08mm, F.Cu at (32.8, 117.8)
- added J1: Vin, lib_fp:TerminalBlock_bornier-2_P5.08mm, F.Cu at (97.9, 59.1)
- added J2: PWM_out, lib_fp:TerminalBlock_bornier-3_P5.08mm, F.Cu at (126.4, 162.8)
- added J2: PWM_out, lib_fp:TerminalBlock_bornier-3_P5.08mm, F.Cu at (262.3, 45.4)
- added J2: PWM_out, lib_fp:TerminalBlock_bornier-3_P5.08mm, F.Cu at (194.0, 45.4)
- added J2: PWM_out, lib_fp:TerminalBlock_bornier-3_P5.08mm, F.Cu at (60.8, 45.5)
- added J2: PWM_out, lib_fp:TerminalBlock_bornier-3_P5.08mm, F.Cu at (193.3, 162.9)
- added J2: PWM_out, lib_fp:TerminalBlock_bornier-3_P5.08mm, F.Cu at (261.6, 162.9)
- added J2: PWM_out, lib_fp:TerminalBlock_bornier-3_P5.08mm, F.Cu at (60.1, 163.0)
- added J2: PWM_out, lib_fp:TerminalBlock_bornier-3_P5.08mm, F.Cu at (128.3, 103.8)
- added J2: PWM_out, lib_fp:TerminalBlock_bornier-3_P5.08mm, F.Cu at (195.2, 103.9)
- added J2: PWM_out, lib_fp:TerminalBlock_bornier-3_P5.08mm, F.Cu at (263.5, 103.9)
- added J2: PWM_out, lib_fp:TerminalBlock_bornier-3_P5.08mm, F.Cu at (62.0, 104.0)
- added J2: PWM_out, lib_fp:TerminalBlock_bornier-3_P5.08mm, F.Cu at (127.1, 45.3)
- added R1: 10k, lib_fp:R_Axial_DIN0207_L6.3mm_D2.5mm_P10.16mm_Horizontal, F.Cu at (234.6, 161.3)
- added R1: 10k, lib_fp:R_Axial_DIN0207_L6.3mm_D2.5mm_P10.16mm_Horizontal, F.Cu at (235.3, 43.8)
- added R1: 10k, lib_fp:R_Axial_DIN0207_L6.3mm_D2.5mm_P10.16mm_Horizontal, F.Cu at (167.0, 43.8)
- added R1: 10k, lib_fp:R_Axial_DIN0207_L6.3mm_D2.5mm_P10.16mm_Horizontal, F.Cu at (33.8, 44.0)
- added R1: 10k, lib_fp:R_Axial_DIN0207_L6.3mm_D2.5mm_P10.16mm_Horizontal, F.Cu at (166.4, 161.3)
- added R1: 10k, lib_fp:R_Axial_DIN0207_L6.3mm_D2.5mm_P10.16mm_Horizontal, F.Cu at (99.4, 161.2)
- added R1: 10k, lib_fp:R_Axial_DIN0207_L6.3mm_D2.5mm_P10.16mm_Horizontal, F.Cu at (33.1, 161.5)
- added R1: 10k, lib_fp:R_Axial_DIN0207_L6.3mm_D2.5mm_P10.16mm_Horizontal, F.Cu at (236.5, 102.3)
- added R1: 10k, lib_fp:R_Axial_DIN0207_L6.3mm_D2.5mm_P10.16mm_Horizontal, F.Cu at (168.2, 102.3)
- added R1: 10k, lib_fp:R_Axial_DIN0207_L6.3mm_D2.5mm_P10.16mm_Horizontal, F.Cu at (101.3, 102.2)
- added R1: 10k, lib_fp:R_Axial_DIN0207_L6.3mm_D2.5mm_P10.16mm_Horizontal, F.Cu at (35.0, 102.4)
- added R1: 10k, lib_fp:R_Axial_DIN0207_L6.3mm_D2.5mm_P10.16mm_Horizontal, F.Cu at (100.1, 43.7)
- added R2: 10k, lib_fp:R_Axial_DIN0207_L6.3mm_D2.5mm_P10.16mm_Horizontal, F.Cu at (238.1, 151.1)
- added R2: 10k, lib_fp:R_Axial_DIN0207_L6.3mm_D2.5mm_P10.16mm_Horizontal, F.Cu at (238.8, 33.6)
- added R2: 10k, lib_fp:R_Axial_DIN0207_L6.3mm_D2.5mm_P10.16mm_Horizontal, F.Cu at (170.5, 33.6)
- added R2: 10k, lib_fp:R_Axial_DIN0207_L6.3mm_D2.5mm_P10.16mm_Horizontal, F.Cu at (37.3, 33.8)
- added R2: 10k, lib_fp:R_Axial_DIN0207_L6.3mm_D2.5mm_P10.16mm_Horizontal, F.Cu at (169.9, 151.1)
- added R2: 10k, lib_fp:R_Axial_DIN0207_L6.3mm_D2.5mm_P10.16mm_Horizontal, F.Cu at (102.9, 151.0)
- added R2: 10k, lib_fp:R_Axial_DIN0207_L6.3mm_D2.5mm_P10.16mm_Horizontal, F.Cu at (36.6, 151.3)
- added R2: 10k, lib_fp:R_Axial_DIN0207_L6.3mm_D2.5mm_P10.16mm_Horizontal, F.Cu at (240.0, 92.1)
- added R2: 10k, lib_fp:R_Axial_DIN0207_L6.3mm_D2.5mm_P10.16mm_Horizontal, F.Cu at (171.7, 92.1)
- added R2: 10k, lib_fp:R_Axial_DIN0207_L6.3mm_D2.5mm_P10.16mm_Horizontal, F.Cu at (104.8, 92.0)
- added R2: 10k, lib_fp:R_Axial_DIN0207_L6.3mm_D2.5mm_P10.16mm_Horizontal, F.Cu at (38.5, 92.2)
- added R2: 10k, lib_fp:R_Axial_DIN0207_L6.3mm_D2.5mm_P10.16mm_Horizontal, F.Cu at (103.6, 33.5)
- added R3: 1k, lib_fp:R_Axial_DIN0207_L6.3mm_D2.5mm_P10.16mm_Horizontal, F.Cu at (53.8, 147.6)
- added R3: 1k, lib_fp:R_Axial_DIN0207_L6.3mm_D2.5mm_P10.16mm_Horizontal, F.Cu at (187.7, 30.0)
- added R3: 1k, lib_fp:R_Axial_DIN0207_L6.3mm_D2.5mm_P10.16mm_Horizontal, F.Cu at (256.0, 30.0)
- added R3: 1k, lib_fp:R_Axial_DIN0207_L6.3mm_D2.5mm_P10.16mm_Horizontal, F.Cu at (54.5, 30.1)
- added R3: 1k, lib_fp:R_Axial_DIN0207_L6.3mm_D2.5mm_P10.16mm_Horizontal, F.Cu at (187.0, 147.5)
- added R3: 1k, lib_fp:R_Axial_DIN0207_L6.3mm_D2.5mm_P10.16mm_Horizontal, F.Cu at (120.1, 147.4)
- added R3: 1k, lib_fp:R_Axial_DIN0207_L6.3mm_D2.5mm_P10.16mm_Horizontal, F.Cu at (255.3, 147.5)
- added R3: 1k, lib_fp:R_Axial_DIN0207_L6.3mm_D2.5mm_P10.16mm_Horizontal, F.Cu at (55.7, 88.6)
- added R3: 1k, lib_fp:R_Axial_DIN0207_L6.3mm_D2.5mm_P10.16mm_Horizontal, F.Cu at (188.9, 88.5)
- added R3: 1k, lib_fp:R_Axial_DIN0207_L6.3mm_D2.5mm_P10.16mm_Horizontal, F.Cu at (122.0, 88.4)
- added R3: 1k, lib_fp:R_Axial_DIN0207_L6.3mm_D2.5mm_P10.16mm_Horizontal, F.Cu at (257.2, 88.5)
- added R3: 1k, lib_fp:R_Axial_DIN0207_L6.3mm_D2.5mm_P10.16mm_Horizontal, F.Cu at (120.8, 29.9)
- added R4: 1k, lib_fp:R_Axial_DIN0207_L6.3mm_D2.5mm_P10.16mm_Horizontal, F.Cu at (40.1, 161.4)
- added R4: 1k, lib_fp:R_Axial_DIN0207_L6.3mm_D2.5mm_P10.16mm_Horizontal, F.Cu at (174.0, 43.7)
- added R4: 1k, lib_fp:R_Axial_DIN0207_L6.3mm_D2.5mm_P10.16mm_Horizontal, F.Cu at (242.3, 43.7)
- added R4: 1k, lib_fp:R_Axial_DIN0207_L6.3mm_D2.5mm_P10.16mm_Horizontal, F.Cu at (40.8, 43.9)
- added R4: 1k, lib_fp:R_Axial_DIN0207_L6.3mm_D2.5mm_P10.16mm_Horizontal, F.Cu at (241.6, 161.2)
- added R4: 1k, lib_fp:R_Axial_DIN0207_L6.3mm_D2.5mm_P10.16mm_Horizontal, F.Cu at (106.4, 161.1)
- added R4: 1k, lib_fp:R_Axial_DIN0207_L6.3mm_D2.5mm_P10.16mm_Horizontal, F.Cu at (173.3, 161.2)
- added R4: 1k, lib_fp:R_Axial_DIN0207_L6.3mm_D2.5mm_P10.16mm_Horizontal, F.Cu at (42.0, 102.4)
- added R4: 1k, lib_fp:R_Axial_DIN0207_L6.3mm_D2.5mm_P10.16mm_Horizontal, F.Cu at (243.5, 102.2)
- added R4: 1k, lib_fp:R_Axial_DIN0207_L6.3mm_D2.5mm_P10.16mm_Horizontal, F.Cu at (108.3, 102.1)
- added R4: 1k, lib_fp:R_Axial_DIN0207_L6.3mm_D2.5mm_P10.16mm_Horizontal, F.Cu at (175.2, 102.2)
- added R4: 1k, lib_fp:R_Axial_DIN0207_L6.3mm_D2.5mm_P10.16mm_Horizontal, F.Cu at (107.1, 43.6)
- added R5: 330, lib_fp:R_Axial_DIN0207_L6.3mm_D2.5mm_P10.16mm_Horizontal, F.Cu at (40.1, 163.9)
- added R5: 330, lib_fp:R_Axial_DIN0207_L6.3mm_D2.5mm_P10.16mm_Horizontal, F.Cu at (174.0, 46.2)
- added R5: 330, lib_fp:R_Axial_DIN0207_L6.3mm_D2.5mm_P10.16mm_Horizontal, F.Cu at (242.3, 46.2)
- added R5: 330, lib_fp:R_Axial_DIN0207_L6.3mm_D2.5mm_P10.16mm_Horizontal, F.Cu at (40.8, 46.4)
- added R5: 330, lib_fp:R_Axial_DIN0207_L6.3mm_D2.5mm_P10.16mm_Horizontal, F.Cu at (241.6, 163.7)
- added R5: 330, lib_fp:R_Axial_DIN0207_L6.3mm_D2.5mm_P10.16mm_Horizontal, F.Cu at (106.4, 163.7)
- added R5: 330, lib_fp:R_Axial_DIN0207_L6.3mm_D2.5mm_P10.16mm_Horizontal, F.Cu at (173.3, 163.7)
- added R5: 330, lib_fp:R_Axial_DIN0207_L6.3mm_D2.5mm_P10.16mm_Horizontal, F.Cu at (42.0, 104.9)
- added R5: 330, lib_fp:R_Axial_DIN0207_L6.3mm_D2.5mm_P10.16mm_Horizontal, F.Cu at (243.5, 104.7)
- added R5: 330, lib_fp:R_Axial_DIN0207_L6.3mm_D2.5mm_P10.16mm_Horizontal, F.Cu at (108.3, 104.7)
- added R5: 330, lib_fp:R_Axial_DIN0207_L6.3mm_D2.5mm_P10.16mm_Horizontal, F.Cu at (175.2, 104.7)
- added R5: 330, lib_fp:R_Axial_DIN0207_L6.3mm_D2.5mm_P10.16mm_Horizontal, F.Cu at (107.1, 46.2)
- added R6: 1k, lib_fp:R_Axial_DIN0207_L6.3mm_D2.5mm_P10.16mm_Horizontal, F.Cu at (128.7, 177.4)
- added R6: 1k, lib_fp:R_Axial_DIN0207_L6.3mm_D2.5mm_P10.16mm_Horizontal, F.Cu at (264.6, 60.0)
- added R6: 1k, lib_fp:R_Axial_DIN0207_L6.3mm_D2.5mm_P10.16mm_Horizontal, F.Cu at (196.3, 60.0)
- added R6: 1k, lib_fp:R_Axial_DIN0207_L6.3mm_D2.5mm_P10.16mm_Horizontal, F.Cu at (63.1, 60.2)
- added R6: 1k, lib_fp:R_Axial_DIN0207_L6.3mm_D2.5mm_P10.16mm_Horizontal, F.Cu at (263.9, 177.5)
- added R6: 1k, lib_fp:R_Axial_DIN0207_L6.3mm_D2.5mm_P10.16mm_Horizontal, F.Cu at (195.7, 177.5)
- added R6: 1k, lib_fp:R_Axial_DIN0207_L6.3mm_D2.5mm_P10.16mm_Horizontal, F.Cu at (62.4, 177.7)
- added R6: 1k, lib_fp:R_Axial_DIN0207_L6.3mm_D2.5mm_P10.16mm_Horizontal, F.Cu at (130.6, 118.4)
- added R6: 1k, lib_fp:R_Axial_DIN0207_L6.3mm_D2.5mm_P10.16mm_Horizontal, F.Cu at (265.8, 118.5)
- added R6: 1k, lib_fp:R_Axial_DIN0207_L6.3mm_D2.5mm_P10.16mm_Horizontal, F.Cu at (197.5, 118.5)
- added R6: 1k, lib_fp:R_Axial_DIN0207_L6.3mm_D2.5mm_P10.16mm_Horizontal, F.Cu at (64.3, 118.7)
- added R6: 1k, lib_fp:R_Axial_DIN0207_L6.3mm_D2.5mm_P10.16mm_Horizontal, F.Cu at (129.4, 59.9)
- added R7: 100, lib_fp:R_Axial_DIN0207_L6.3mm_D2.5mm_P10.16mm_Horizontal, F.Cu at (58.5, 177.6)
- added R7: 100, lib_fp:R_Axial_DIN0207_L6.3mm_D2.5mm_P10.16mm_Horizontal, F.Cu at (192.4, 60.0)
- added R7: 100, lib_fp:R_Axial_DIN0207_L6.3mm_D2.5mm_P10.16mm_Horizontal, F.Cu at (260.7, 60.0)
- added R7: 100, lib_fp:R_Axial_DIN0207_L6.3mm_D2.5mm_P10.16mm_Horizontal, F.Cu at (59.2, 60.1)
- added R7: 100, lib_fp:R_Axial_DIN0207_L6.3mm_D2.5mm_P10.16mm_Horizontal, F.Cu at (260.0, 177.5)
- added R7: 100, lib_fp:R_Axial_DIN0207_L6.3mm_D2.5mm_P10.16mm_Horizontal, F.Cu at (124.8, 177.4)
- added R7: 100, lib_fp:R_Axial_DIN0207_L6.3mm_D2.5mm_P10.16mm_Horizontal, F.Cu at (191.7, 177.5)
- added R7: 100, lib_fp:R_Axial_DIN0207_L6.3mm_D2.5mm_P10.16mm_Horizontal, F.Cu at (60.4, 118.6)
- added R7: 100, lib_fp:R_Axial_DIN0207_L6.3mm_D2.5mm_P10.16mm_Horizontal, F.Cu at (261.9, 118.5)
- added R7: 100, lib_fp:R_Axial_DIN0207_L6.3mm_D2.5mm_P10.16mm_Horizontal, F.Cu at (126.7, 118.4)
- added R7: 100, lib_fp:R_Axial_DIN0207_L6.3mm_D2.5mm_P10.16mm_Horizontal, F.Cu at (193.6, 118.5)
- added R7: 100, lib_fp:R_Axial_DIN0207_L6.3mm_D2.5mm_P10.16mm_Horizontal, F.Cu at (125.5, 59.9)
- added R8: 1k, lib_fp:R_Axial_DIN0207_L6.3mm_D2.5mm_P10.16mm_Horizontal, F.Cu at (29.5, 161.3)
- added R8: 1k, lib_fp:R_Axial_DIN0207_L6.3mm_D2.5mm_P10.16mm_Horizontal, F.Cu at (163.4, 43.7)
- added R8: 1k, lib_fp:R_Axial_DIN0207_L6.3mm_D2.5mm_P10.16mm_Horizontal, F.Cu at (231.7, 43.7)
- added R8: 1k, lib_fp:R_Axial_DIN0207_L6.3mm_D2.5mm_P10.16mm_Horizontal, F.Cu at (30.2, 43.8)
- added R8: 1k, lib_fp:R_Axial_DIN0207_L6.3mm_D2.5mm_P10.16mm_Horizontal, F.Cu at (95.8, 161.1)
- added R8: 1k, lib_fp:R_Axial_DIN0207_L6.3mm_D2.5mm_P10.16mm_Horizontal, F.Cu at (231.0, 161.2)
- added R8: 1k, lib_fp:R_Axial_DIN0207_L6.3mm_D2.5mm_P10.16mm_Horizontal, F.Cu at (162.8, 161.2)
- added R8: 1k, lib_fp:R_Axial_DIN0207_L6.3mm_D2.5mm_P10.16mm_Horizontal, F.Cu at (31.4, 102.3)
- added R8: 1k, lib_fp:R_Axial_DIN0207_L6.3mm_D2.5mm_P10.16mm_Horizontal, F.Cu at (97.7, 102.1)
- added R8: 1k, lib_fp:R_Axial_DIN0207_L6.3mm_D2.5mm_P10.16mm_Horizontal, F.Cu at (232.9, 102.2)
- added R8: 1k, lib_fp:R_Axial_DIN0207_L6.3mm_D2.5mm_P10.16mm_Horizontal, F.Cu at (164.6, 102.2)
- added R8: 1k, lib_fp:R_Axial_DIN0207_L6.3mm_D2.5mm_P10.16mm_Horizontal, F.Cu at (96.5, 43.6)
- added RV1: 10k, lib_fp:Potentiometer_Bourns_3266Y_Vertical, F.Cu at (57.8, 147.0)
- added RV1: 10k, lib_fp:Potentiometer_Bourns_3266Y_Vertical, F.Cu at (191.7, 29.3)
- added RV1: 10k, lib_fp:Potentiometer_Bourns_3266Y_Vertical, F.Cu at (259.9, 29.3)
- added RV1: 10k, lib_fp:Potentiometer_Bourns_3266Y_Vertical, F.Cu at (58.4, 29.5)
- added RV1: 10k, lib_fp:Potentiometer_Bourns_3266Y_Vertical, F.Cu at (259.3, 146.8)
- added RV1: 10k, lib_fp:Potentiometer_Bourns_3266Y_Vertical, F.Cu at (124.1, 146.7)
- added RV1: 10k, lib_fp:Potentiometer_Bourns_3266Y_Vertical, F.Cu at (191.0, 146.8)
- added RV1: 10k, lib_fp:Potentiometer_Bourns_3266Y_Vertical, F.Cu at (59.6, 88.0)
- added RV1: 10k, lib_fp:Potentiometer_Bourns_3266Y_Vertical, F.Cu at (261.1, 87.8)
- added RV1: 10k, lib_fp:Potentiometer_Bourns_3266Y_Vertical, F.Cu at (125.9, 87.7)
- added RV1: 10k, lib_fp:Potentiometer_Bourns_3266Y_Vertical, F.Cu at (192.9, 87.8)
- added RV1: 10k, lib_fp:Potentiometer_Bourns_3266Y_Vertical, F.Cu at (124.7, 29.2)
- added RV2: 250k, lib_fp:Potentiometer_Bourns_3266Y_Vertical, F.Cu at (44.4, 176.3)
- added RV2: 250k, lib_fp:Potentiometer_Bourns_3266Y_Vertical, F.Cu at (178.3, 58.7)
- added RV2: 250k, lib_fp:Potentiometer_Bourns_3266Y_Vertical, F.Cu at (246.6, 58.7)
- added RV2: 250k, lib_fp:Potentiometer_Bourns_3266Y_Vertical, F.Cu at (45.1, 58.8)
- added RV2: 250k, lib_fp:Potentiometer_Bourns_3266Y_Vertical, F.Cu at (245.9, 176.2)
- added RV2: 250k, lib_fp:Potentiometer_Bourns_3266Y_Vertical, F.Cu at (177.6, 176.2)
- added RV2: 250k, lib_fp:Potentiometer_Bourns_3266Y_Vertical, F.Cu at (110.7, 176.1)
- added RV2: 250k, lib_fp:Potentiometer_Bourns_3266Y_Vertical, F.Cu at (46.3, 117.3)
- added RV2: 250k, lib_fp:Potentiometer_Bourns_3266Y_Vertical, F.Cu at (247.8, 117.2)
- added RV2: 250k, lib_fp:Potentiometer_Bourns_3266Y_Vertical, F.Cu at (179.5, 117.2)
- added RV2: 250k, lib_fp:Potentiometer_Bourns_3266Y_Vertical, F.Cu at (112.6, 117.1)
- added RV2: 250k, lib_fp:Potentiometer_Bourns_3266Y_Vertical, F.Cu at (111.4, 58.6)
- added U1: SG3525, lib_fp:DIP-16_W7.62mm_LongPads, F.Cu at (44.7, 151.2)
- added U1: SG3525, lib_fp:DIP-16_W7.62mm_LongPads, F.Cu at (178.6, 33.5)
- added U1: SG3525, lib_fp:DIP-16_W7.62mm_LongPads, F.Cu at (246.8, 33.5)
- added U1: SG3525, lib_fp:DIP-16_W7.62mm_LongPads, F.Cu at (45.3, 33.7)
- added U1: SG3525, lib_fp:DIP-16_W7.62mm_LongPads, F.Cu at (246.2, 151.0)
- added U1: SG3525, lib_fp:DIP-16_W7.62mm_LongPads, F.Cu at (177.9, 151.0)
- added U1: SG3525, lib_fp:DIP-16_W7.62mm_LongPads, F.Cu at (111.0, 151.0)
- added U1: SG3525, lib_fp:DIP-16_W7.62mm_LongPads, F.Cu at (46.6, 92.2)
- added U1: SG3525, lib_fp:DIP-16_W7.62mm_LongPads, F.Cu at (248.1, 92.0)
- added U1: SG3525, lib_fp:DIP-16_W7.62mm_LongPads, F.Cu at (179.8, 92.0)
- added U1: SG3525, lib_fp:DIP-16_W7.62mm_LongPads, F.Cu at (112.8, 92.0)
- added U1: SG3525, lib_fp:DIP-16_W7.62mm_LongPads, F.Cu at (111.6, 33.5)
Routing:
- net (no net): track 3342.7 -> 3355.7 mm
Other:
- board size 231.5 x 153.5 mm -> 243.7 x 155.2 mm
- board text added: "+15V"
