File: Electronica de Potencia/TP's/TPN3/PCB/Transistores/MOSFET-IGBT/MOSFET-IGBT.sch (KiCad schematic (older format))
At the start: 17 parts, among them J1 Vin, J2 PWM_IN, Q1 FGPF7N60RUFD, Q2 IRF840, T1 50:50

Commit message: Termino placa 3 de potencia
Parts:
- added G1: logo, lib_fp:logo_utn_fsilk_small, symbol MOSFET-IGBT:logo
- added HS1, HS2: Heatsink, lib_fp:Heatsink_TO220_A, symbol MOSFET-IGBT:Heatsink
- D1, D2, D3, D4: footprint Diode_THT:D_DO-35_SOD27_P7.62mm_Horizontal -> lib_fp:D_DO-34_SOD68_P7.62mm_Horizontal; symbol Diode:1N4148 -> MOSFET-IGBT:1N4148
- J1: footprint (none) -> lib_fp:TerminalBlock_bornier-2_P5.08mm; symbol Connector:Screw_Terminal_01x02 -> MOSFET-IGBT:Screw_Terminal_01x02
- J2: footprint (none) -> lib_fp:TerminalBlock_bornier-3_P5.08mm; symbol Connector:Screw_Terminal_01x03 -> MOSFET-IGBT:Screw_Terminal_01x03
- JP1, JP3: footprint (none) -> lib_fp:PinHeader_1x02_P2.54mm_Vertical; symbol Device:Jumper_NC_Small -> MOSFET-IGBT:Jumper_NC_Small
- JP2: footprint (none) -> lib_fp:PinHeader_1x03_P2.54mm_Vertical; symbol Device:Jumper_NC_Dual -> MOSFET-IGBT:Jumper_NC_Dual
- Q1: footprint (none) -> lib_fp:TO-220-3_Vertical; symbol Device:Q_NIGBT_GCE -> MOSFET-IGBT:Q_NIGBT_GCE
- Q2: footprint Package_DirectFET:DirectFET_MT -> lib_fp:TO-220-3_Vertical; symbol Transistor_FET:IRF8301M -> MOSFET-IGBT:IRF8301M
- R1: footprint (none) -> lib_fp:R_Axial_DIN0207_L6.3mm_D2.5mm_P10.16mm_Horizontal; symbol Device:R_US -> MOSFET-IGBT:R_US
- R2: footprint (none) -> lib_fp:R_Axial_Power_L50.0mm_W9.0mm_P55.88mm; symbol Device:R_US -> MOSFET-IGBT:R_US
- T1: footprint (none) -> lib_fp:Transformador_EE25; symbol Device:Transformer_1P_1S -> MOSFET-IGBT:Transformer_1P_1S
- TP1, TP2, TP3: footprint (none) -> lib_fp:Testpoint; symbol Connector:TestPoint_Probe -> MOSFET-IGBT:TestPoint_Probe
Changed lines of the file:
@@
 EESchema Schematic File Version 4
+LIBS:MOSFET-IGBT-cache
 EELAYER 29 0
 EELAYER END
@@
 $EndDescr
 $Comp
-L Connector:Screw_Terminal_01x03 J2
+L MOSFET-IGBT:Screw_Terminal_01x03 J2
 U 1 1 5CDA3F5E
 P 3150 4250
 F 0 "J2" H 3230 4292 50  0000 L CNN
 F 1 "PWM_IN" H 3230 4201 50  0000 L CNN
-F 2 "" H 3150 4250 50  0001 C CNN
+F 2 "lib_fp:TerminalBlock_bornier-3_P5.08mm" H 3150 4250 50  0001 C CNN
 F 3 "~" H 3150 4250 50  0001 C CNN
 	1    3150 4250
@@
 	2950 4150 2650 4150
 $Comp
-L power:GND #PWR0101
+L MOSFET-IGBT:GND #PWR0101
 U 1 1 5CDA47F5
 P 2650 4250
@@
 	2650 4350 2950 4350
 $Comp
-L Diode:1N4148 D1
+L MOSFET-IGBT:1N4148 D1
 U 1 1 5CDA5C46
 P 4200 3500
 F 0 "D1" V 4154 3579 50  0000 L CNN
 F 1 "1N4148" V 4245 3579 50  0000 L CNN
-F 2 "Diode_THT:D_DO-35_SOD27_P7.62mm_Horizontal" H 4200 3325 50  0001 C CNN
+F 2 "lib_fp:D_DO-34_SOD68_P7.62mm_Horizontal" H 4200 3325 50  0001 C CNN
 F 3 "https://assets.nexperia.com/documents/data-sheet/1N4148_1N4448.pdf" H 4200 3500 50  0001 C CNN
 	1    4200 3500
@@
 $EndComp
 $Comp
-L Diode:1N4148 D2
+L MOSFET-IGBT:1N4148 D2
 U 1 1 5CDA8AD3
 P 4200 4500
 F 0 "D2" V 4154 4579 50  0000 L CNN
 F 1 "1N4148" V 4245 4579 50  0000 L CNN
-F 2 "Diode_THT:D_DO-35_SOD27_P7.62mm_Horizontal" H 4200 4325 50  0001 C CNN
+F 2 "lib_fp:D_DO-34_SOD68_P7.62mm_Horizontal" H 4200 4325 50  0001 C CNN
 F 3 "https://assets.nexperia.com/documents/data-sheet/1N4148_1N4448.pdf" H 4200 4500 50  0001 C CNN
 	1    4200 4500
@@
 $EndComp
 $Comp
-L Diode:1N4148 D3
+L MOSFET-IGBT:1N4148 D3
 U 1 1 5CDAAC55
 P 4750 3500
 F 0 "D3" V 4704 3579 50  0000 L CNN
 F 1 "1N4148" V 4795 3579 50  0000 L CNN
-F 2 "Diode_THT:D_DO-35_SOD27_P7.62mm_Horizontal" H 4750 3325 50  0001 C CNN
+F 2 "lib_fp:D_DO-34_SOD68_P7.62mm_Horizontal" H 4750 3325 50  0001 C CNN
 F 3 "https://assets.nexperia.com/documents/data-sheet/1N4148_1N4448.pdf" H 4750 3500 50  0001 C CNN
 	1    4750 3500
@@
 $EndComp
 $Comp
-L Device:Transformer_1P_1S T1
+L MOSFET-IGBT:Transformer_1P_1S T1
 U 1 1 5CDAD0CD
 P 5400 4000
 F 0 "T1" H 5400 4300 50  0000 C CNN
 F 1 "50:50" H 5400 3750 50  0000 C CNN
-F 2 "" H 5400 4000 50  0001 C CNN
+F 2 "lib_fp:Transformador_EE25" H 5400 4000 50  0001 C CNN
 F 3 "~" H 5400 4000 50  0001 C CNN
 	1    5400 4000
@@
 $EndComp
 $Comp
-L Connector:Screw_Terminal_01x02 J1
+L MOSFET-IGBT:Screw_Terminal_01x02 J1
 U 1 1 5CDAEFEA
 P 3150 3600
 F 0 "J1" H 3230 3592 50  0000 L CNN
 F 1 "Vin" H 3230 3501 50  0000 L CNN
-F 2 "" H 3150 3600 50  0001 C CNN
+F 2 "lib_fp:TerminalBlock_bornier-2_P5.08mm" H 3150 3600 50  0001 C CNN
 F 3 "~" H 3150 3600 50  0001 C CNN
 	1    3150 3600
@@
 $EndComp
 $Comp
-L power:GND #PWR0102
+L MOSFET-IGBT:GND #PWR0102
 U 1 1 5CDAF70A
 P 2900 3750
@@
 	2900 3700 2950 3700
 $Comp
-L power:+15V #PWR0103
+L MOSFET-IGBT:+15V #PWR0103
 U 1 1 5CDB0039
 P 2900 3550
@@
 	2900 3600 2950 3600
 $Comp
-L Diode:1N4148 D4
+L MOSFET-IGBT:1N4148 D4
 U 1 1 5CDB5DA8
 P 4750 4500
 F 0 "D4" V 4704 4579 50  0000 L CNN
 F 1 "1N4148" V 4795 4579 50  0000 L CNN
-F 2 "Diode_THT:D_DO-35_SOD27_P7.62mm_Horizontal" H 4750 4325 50  0001 C CNN
+F 2 "lib_fp:D_DO-34_SOD68_P7.62mm_Horizontal" H 4750 4325 50  0001 C CNN
 F 3 "https://assets.nexperia.com/documents/data-sheet/1N4148_1N4448.pdf" H 4750 4500 50  0001 C CNN
 	1    4750 4500
@@
 	4200 4200 4200 3650
 $Comp
-L power:GND #PWR0104
+L MOSFET-IGBT:GND #PWR0104
 U 1 1 5CDBB0FB
 P 4450 4800
@@
 Connection ~ 4500 3050
 $Comp
-L Device:Q_NIGBT_GCE Q1
+L MOSFET-IGBT:Q_NIGBT_GCE Q1
 U 1 1 5CDBEC5A
 P 6850 3800
 F 0 "Q1" H 7040 3846 50  0000 L CNN
 F 1 "FGPF7N60RUFD " H 7040 3755 50  0000 L CNN
-F 2 "" H 7050 3900 50  0001 C CNN
+F 2 "lib_fp:TO-220-3_Vertical" H 7050 3900 50  0001 C CNN
 F 3 "~" H 6850 3800 50  0001 C CNN
 	1    6850 3800
@@
 $EndComp
 $Comp
-L Device:R_US R1
+L MOSFET-IGBT:R_US R1
 U 1 1 5CDC053C
 P 6300 4000
 F 0 "R1" H 6368 4046 50  0000 L CNN
 F 1 "220" H 6368 3955 50  0000 L CNN
-F 2 "" V 6340 3990 50  0001 C CNN
+F 2 "lib_fp:R_Axial_DIN0207_L6.3mm_D2.5mm_P10.16mm_Horizontal" V 6340 3990 50  0001 C CNN
 F 3 "~" H 6300 4000 50  0001 C CNN
 	1    6300 4000
@@
 $EndComp
 $Comp
-L power:GND #PWR0105
+L MOSFET-IGBT:GND #PWR0105
 U 1 1 5CDC0FF3
 P 6950 4400
@@
 Connection ~ 6950 4200
 $Comp
-L Device:R_US R2
+L MOSFET-IGBT:R_US R2
 U 1 1 5CDC3BAC
 P 7550 2850
 F 0 "R2" H 7618 2896 50  0000 L CNN
 F 1 "15" H 7618 2805 50  0000 L CNN
-F 2 "" V 7590 2840 50  0001 C CNN
+F 2 "lib_fp:R_Axial_Power_L50.0mm_W9.0mm_P55.88mm" V 7590 2840 50  0001 C CNN
 F 3 "~" H 7550 2850 50  0001 C CNN
 	1    7550 2850
@@
 $EndComp
 $Comp
-L Device:Jumper_NC_Dual JP2
+L MOSFET-IGBT:Jumper_NC_Dual JP2
 U 1 1 5CDC4C16
 P 7550 3200
 F 0 "JP2" H 7550 3347 50  0000 C CNN
 F 1 "Jumper_NC_Dual" H 7550 3438 50  0001 C CNN
-F 2 "" H 7550 3200 50  0001 C CNN
+F 2 "lib_fp:PinHeader_1x03_P2.54mm_Vertical" H 7550 3200 50  0001 C CNN
 F 3 "~" H 7550 3200 50  0001 C CNN
 	1    7550 3200
@@
 	6950 3200 7300 3200
 $Comp
-L power:+15V #PWR0106
+L MOSFET-IGBT:+15V #PWR0106
 U 1 1 5CDC63BE
 P 7550 2600
@@
 	7550 2600 7550 2700
 $Comp
-L Device:Jumper_NC_Small JP1
+L MOSFET-IGBT:Jumper_NC_Small JP1
 U 1 1 5CDC7EF0
 P 6500 3800
 F 0 "JP1" H 6500 3921 50  0000 C CNN
 F 1 "Jumper_NC_Small" H 6500 3921 50  0001 C CNN
-F 2 "" H 6500 3800 50  0001 C CNN
+F 2 "lib_fp:PinHeader_1x02_P2.54mm_Vertical" H 6500 3800 50  0001 C CNN
 F 3 "~" H 6500 3800 50  0001 C CNN
 	1    6500 3800
@@
 	6300 3800 6300 3550
 $Comp
-L Transistor_FET:IRF8301M Q2
+L MOSFET-IGBT:IRF8301M Q2
 U 1 1 5CDC9E4F
 P 8000 3800
 F 0 "Q2" H 8206 3846 50  0000 L CNN
 F 1 "IRF840" H 8206 3755 50  0000 L CNN
-F 2 "Package_DirectFET:DirectFET_MT" H 8000 3800 50  0001 C CIN
+F 2 "lib_fp:TO-220-3_Vertical" H 8000 3800 50  0001 C CIN
 F 3 "https://www.infineon.com/dgdl/irf8301mpbf.pdf?fileId=5546d462533600a40153560d0e7a1d58" H 8000 3800 50  0001 L CNN
 	1    8000 3800
@@
 	8100 4200 8100 4000
 $Comp
-L Device:Jumper_NC_Small JP3
+L MOSFET-IGBT:Jumper_NC_Small JP3
 U 1 1 5CDD2019
 P 7700 3800
 F 0 "JP3" H 7700 3921 50  0000 C CNN
 F 1 "Jumper_NC_Small" H 7700 3921 50  0001 C CNN
-F 2 "" H 7700 3800 50  0001 C CNN
+F 2 "lib_fp:PinHeader_1x02_P2.54mm_Vertical" H 7700 3800 50  0001 C CNN
 F 3 "~" H 7700 3800 50  0001 C CNN
 	1    7700 3800
@@
 	6300 3550 7600 3550
 $Comp
-L power:+15V #PWR0107
+L MOSFET-IGBT:+15V #PWR0107
 U 1 1 5CDBA827
 P 4500 2600
@@
 	4500 2600 4500 3050
 $Comp
-L Connector:TestPoint_Probe TP3
+L MOSFET-IGBT:TestPoint_Probe TP3
 U 1 1 5CDF2A14
 P 8100 3450
 F 0 "TP3" H 8253 3551 50  0000 L CNN
 F 1 "TP_VDS" H 8253 3460 50  0000 L CNN
-F 2 "" H 8300 3450 50  0001 C CNN
+F 2 "lib_fp:Testpoint" H 8300 3450 50  0001 C CNN
 F 3 "~" H 8300 3450 50  0001 C CNN
 	1    8100 3450
@@
 	8100 3450 8100 3200
 $Comp
-L Connector:TestPoint_Probe TP1
+L MOSFET-IGBT:TestPoint_Probe TP1
 U 1 1 5CDF4DF4
 P 6300 3800
 F 0 "TP1" H 6550 3950 50  0000 L CNN
 F 1 "TP_VBE_VGS" H 6450 3850 50  0000 L CNN
-F 2 "" H 6500 3800 50  0001 C CNN
+F 2 "lib_fp:Testpoint" H 6500 3800 50  0001 C CNN
 F 3 "~" H 6500 3800 50  0001 C CNN
 	1    6300 3800
@@
 $EndComp
 $Comp
-L Connector:TestPoint_Probe TP2
+L MOSFET-IGBT:TestPoint_Probe TP2
 U 1 1 5CDFA8CD
 P 6950 4200
 F 0 "TP2" H 7102 4301 50  0000 L CNN
 F 1 "GND" H 7102 4210 50  0000 L CNN
-F 2 "" H 7150 4200 50  0001 C CNN
+F 2 "lib_fp:Testpoint" H 7150 4200 50  0001 C CNN
 F 3 "~" H 7150 4200 50  0001 C CNN
 	1    6950 4200
 	1    0    0    -1
 $EndComp
+$Comp
+L MOSFET-IGBT:Heatsink HS1
+U 1 1 5CE3BEC6
+P 8750 3875
+F 0 "HS1" H 8892 3996 50  0000 L CNN
+F 1 "Heatsink" H 8892 3905 50  0000 L CNN
+F 2 "lib_fp:Heatsink_TO220_A" H 8762 3875 50  0001 C CNN
+F 3 "" H 8762 3875 50  0001 C CNN
+	1    8750 3875
+	1    0    0    -1
+$EndComp
+$Comp
+L MOSFET-IGBT:Heatsink HS2
+U 1 1 5CE3D568
+P 9400 3875
+F 0 "HS2" H 9542 3996 50  0000 L CNN
+F 1 "Heatsink" H 9542 3905 50  0000 L CNN
+F 2 "lib_fp:Heatsink_TO220_A" H 9412 3875 50  0001 C CNN
+F 3 "" H 9412 3875 50  0001 C CNN
+	1    9400 3875
+	1    0    0    -1
+$EndComp
+$Comp
+L MOSFET-IGBT:logo G1
+U 1 1 5CE3E2E6
+P 8700 4125
+F 0 "G1" H 8776 4125 60  0000 L CNN
+F 1 "logo" H 8700 4155 60  0001 C CNN
+F 2 "lib_fp:logo_utn_fsilk_small" H 8700 4125 50  0001 C CNN
+F 3 "" H 8700 4125 50  0001 C CNN
+	1    8700 4125
+	1    0    0    -1
+$EndComp
