File: Electronica de Potencia/TP's/TPN3/PCB/Transistores/MOSFET-IGBT/MOSFET-IGBT.kicad_pcb (KiCad board)
At the start: 2 copper layers, 70.9 x 52.3 mm, 20 parts, among them J1 Vin, J2 PWM_IN, Q1 FGPF7N60RUFD, Q2 IRF840, T1 50:50

Commit message: Actualizo placa MOSFET_IGBT de potencia
Parts:
- JP1: value Jumper_NC_Small -> IGBT
- JP2: value Jumper_NC_Dual -> MOSFET O IGBT
- JP3: value Jumper_NC_Small -> MOSFET
Routing:
- net Net-(JP2-Pad3): track 77.5 -> 81.3 mm
Changed lines of the file:
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@@
     (mod_text_size 1 1)
     (mod_text_width 0.15)
-    (pad_size 2 4)
-    (pad_drill 1.1)
+    (pad_size 4 4)
+    (pad_drill 1.2)
     (pad_to_mask_clearance 0.051)
     (solder_mask_min_width 0.25)
@@
       (effects (font (size 1 1) (thickness 0.15)))
     )
-    (fp_text value Heatsink (at 10 22 270) (layer F.Fab)
+    (fp_text value Heatsink (at 9.8298 17.7546 270) (layer F.Fab)
       (effects (font (size 1 1) (thickness 0.15)))
     )
@@
       (effects (font (size 1 1) (thickness 0.15)))
     )
-    (fp_text value Heatsink (at 10 22 270) (layer F.Fab)
+    (fp_text value Heatsink (at 9.7536 17.399 270) (layer F.Fab)
       (effects (font (size 1 1) (thickness 0.15)))
     )
@@
       (effects (font (size 1 1) (thickness 0.15)))
     )
-    (fp_text value 220 (at 5.08 2.37) (layer F.Fab)
+    (fp_text value 220 (at 6.4008 -0.0762) (layer F.Fab)
       (effects (font (size 1 1) (thickness 0.15)))
     )
@@
     (fp_line (start 11.21 1.5) (end 11.21 -1.5) (layer F.CrtYd) (width 0.05))
     (fp_line (start 11.21 -1.5) (end -1.05 -1.5) (layer F.CrtYd) (width 0.05))
-    (fp_text user %R (at 5.08 0) (layer F.Fab)
-      (effects (font (size 1 1) (thickness 0.15)))
-    )
-    (pad 1 thru_hole circle (at 0 0) (size 1.6 1.6) (drill 0.8) (layers *.Cu *.Mask)
+    (fp_text user %R (at 3.1242 -0.0508) (layer F.Fab)
+      (effects (font (size 1 1) (thickness 0.15)))
+    )
+    (pad 1 thru_hole circle (at 0 0) (size 2 2) (drill 0.8) (layers *.Cu *.Mask)
       (net 5 "Net-(JP1-Pad1)"))
-    (pad 2 thru_hole oval (at 10.16 0) (size 1.6 1.6) (drill 0.8) (layers *.Cu *.Mask)
+    (pad 2 thru_hole oval (at 10.16 0) (size 2 2) (drill 0.8) (layers *.Cu *.Mask)
       (net 3 GND))
     (model ${KISYS3DMOD}/Resistor_THT.3dshapes/R_Axial_DIN0207_L6.3mm_D2.5mm_P10.16mm_Horizontal.wrl
@@
       (effects (font (size 1 1) (thickness 0.15)))
     )
-    (fp_text value 15 (at 27.94 5.62) (layer F.Fab)
+    (fp_text value 15 (at 31.9532 0.1016) (layer F.Fab)
       (effects (font (size 1 1) (thickness 0.15)))
     )
@@
       (effects (font (size 1 1) (thickness 0.15)))
     )
-    (pad 1 thru_hole circle (at 0 0) (size 2.4 2.4) (drill 1.2) (layers *.Cu *.Mask)
+    (pad 1 thru_hole circle (at 0 0) (size 4 4) (drill 1.2) (layers *.Cu *.Mask)
       (net 1 +15V))
-    (pad 2 thru_hole oval (at 55.88 0) (size 2.4 2.4) (drill 1.2) (layers *.Cu *.Mask)
+    (pad 2 thru_hole oval (at 55.88 0) (size 4 4) (drill 1.2) (layers *.Cu *.Mask)
       (net 8 "Net-(JP2-Pad2)"))
     (model ${KISYS3DMOD}/Resistor_THT.3dshapes/R_Axial_Power_L50.0mm_W9.0mm_P55.88mm.wrl
@@
       (effects (font (size 1 1) (thickness 0.15)))
     )
-    (fp_text value TP_VBE_VGS (at 0 2.33) (layer F.Fab)
+    (fp_text value TP_VBE_VGS (at 0 2.8702) (layer F.Fab)
       (effects (font (size 1 1) (thickness 0.15)))
     )
@@
       (effects (font (size 1 1) (thickness 0.15)))
     )
-    (fp_text value 50:50 (at 15.62 23.72 270) (layer F.Fab)
+    (fp_text value 50:50 (at 16.3576 11.2014) (layer F.Fab)
       (effects (font (size 1 1) (thickness 0.15)))
     )
@@
       (effects (font (size 1 1) (thickness 0.15)))
     )
-    (fp_text value Jumper_NC_Small (at 0 4.87) (layer F.Fab)
+    (fp_text value IGBT (at -3.4544 1.143 90) (layer F.Fab)
       (effects (font (size 1 1) (thickness 0.15)))
     )
@@
       (effects (font (size 1 1) (thickness 0.15)))
     )
-    (fp_text value Jumper_NC_Dual (at 0 7.41) (layer F.Fab)
+    (fp_text value "MOSFET O IGBT" (at -3.048 1.905 90) (layer F.Fab)
       (effects (font (size 1 1) (thickness 0.15)))
     )
@@
       (effects (font (size 1 1) (thickness 0.15)))
     )
-    (fp_text value Jumper_NC_Small (at 0 4.87 180) (layer F.Fab)
+    (fp_text value MOSFET (at 3.4036 1.2192 270) (layer F.Fab)
       (effects (font (size 1 1) (thickness 0.15)))
     )
@@
   (segment (start 132.334 166.116) (end 132.334 166.243) (width 2) (layer B.Cu) (net 8))
   (segment (start 132.334 166.243) (end 134.493 166.243) (width 2) (layer B.Cu) (net 8))
-  (segment (start 136.652 169.291) (end 139.573 166.37) (width 2) (layer B.Cu) (net 9))
-  (segment (start 131.445 169.291) (end 136.652 169.291) (width 2) (layer B.Cu) (net 9))
-  (segment (start 125.73 158.496) (end 125.73 163.576) (width 2) (layer B.Cu) (net 9))
-  (segment (start 125.73 163.576) (end 131.445 169.291) (width 2) (layer B.Cu) (net 9))
   (segment (start 139.573 135.573) (end 139.573 136.525) (width 2) (layer B.Cu) (net 9))
-  (segment (start 139.573 166.37) (end 139.573 136.525) (width 2) (layer B.Cu) (net 9))
   (segment (start 139.573 136.525) (end 139.573 135.192) (width 2) (layer B.Cu) (net 9))
   (segment (start 133.548 124.206) (end 139.573 130.231) (width 2) (layer B.Cu) (net 9))
@@
   (segment (start 139.573 130.231) (end 139.573 133.477) (width 2) (layer B.Cu) (net 9))
   (segment (start 139.573 133.477) (end 139.573 135.192) (width 2) (layer B.Cu) (net 9))
+  (segment (start 139.573 169.0116) (end 139.573 136.525) (width 2) (layer B.Cu) (net 9))
+  (segment (start 138.1252 170.4594) (end 139.573 169.0116) (width 2) (layer B.Cu) (net 9))
+  (segment (start 130.3528 170.4594) (end 138.1252 170.4594) (width 2) (layer B.Cu) (net 9))
+  (segment (start 125.73 158.496) (end 125.73 165.8366) (width 2) (layer B.Cu) (net 9))
+  (segment (start 125.73 165.8366) (end 130.3528 170.4594) (width 2) (layer B.Cu) (net 9))
   (segment (start 128.778 130.81) (end 133.731 130.81) (width 2) (layer B.Cu) (net 10))
   (segment (start 125.73 133.858) (end 128.778 130.81) (width 2) (layer B.Cu) (net 10))
