File: Electronica de Potencia/TP's/TPN3/PCB/Transistores/[Kicad] MOSFET-IGBT/MOSFET-IGBT.sch (KiCad schematic (older format))
At the start: 20 parts, among them J1 Vin, J2 PWM_IN, Q1 FGPF7N60RUFD, Q2 IRF840, T1 50:50

Commit message: Arreglo placa de potencia
Parts:
- TP3: value TP_VDS -> TP_VCE_VDS
Connections:
- net GND: no longer Q1.3 (E), Q2.3 (S), R1.2, T1.3 (SA), TP2.1
- net PWM_A: now also J2.3 (Pin_3); no longer J2.1 (Pin_1)
- net PWM_B: now also J2.1 (Pin_1); no longer J2.3 (Pin_3)
- net at JP2.2, R2.2: now also TP3.1
- net at JP2.3, Q2.1 (D): no longer TP3.1
- new net Earth: Q1.3 (E), Q2.3 (S), R1.2, T1.3 (SA), TP2.1
Other:
- note added: "unir masas"
- moved on the sheet: JP1, JP2, JP3, Q1, Q2, R1, R2, TP1, TP2, TP3
Changed lines of the file:
@@
 	1    0    0    -1
 $EndComp
+Text Label 2650 4400 2    50   ~ 0
+PWM_A
 Text Label 2650 4150 2    50   ~ 0
-PWM_A
-Text Label 2650 4400 2    50   ~ 0
 PWM_B
 Wire Wire Line
@@
 	4750 3800 3800 3800
 Connection ~ 4750 3800
-Text Label 3800 3800 2    50   ~ 0
-PWM_A
 Wire Wire Line
 	4750 4350 4750 3800
 Wire Wire Line
 	5000 4200 4200 4200
-Text Label 3800 4200 2    50   ~ 0
-PWM_B
 Wire Wire Line
 	4200 4350 4200 4200
@@
 Wire Wire Line
 	4200 4200 4200 3650
-$Comp
-L MOSFET-IGBT:GND #PWR0104
-U 1 1 5CDBB0FB
-P 4450 4800
-F 0 "#PWR0104" H 4450 4550 50  0001 C CNN
-F 1 "GND" H 4455 4627 50  0000 C CNN
-F 2 "" H 4450 4800 50  0001 C CNN
-F 3 "" H 4450 4800 50  0001 C CNN
-	1    4450 4800
-	1    0    0    -1
-$EndComp
-Wire Wire Line
-	4450 4800 4200 4800
 Wire Wire Line
 	4200 4800 4200 4650
 Wire Wire Line
-	4450 4800 4750 4800
-Wire Wire Line
 	4750 4800 4750 4650
-Connection ~ 4450 4800
 Wire Wire Line
 	4500 3050 4200 3050
@@
 L MOSFET-IGBT:Q_NIGBT_GCE Q1
 U 1 1 5CDBEC5A
-P 6850 3800
-F 0 "Q1" H 7040 3846 50  0000 L CNN
-F 1 "FGPF7N60RUFD " H 7040 3755 50  0000 L CNN
-F 2 "lib_fp:TO-220-3_Vertical" H 7050 3900 50  0001 C CNN
-F 3 "~" H 6850 3800 50  0001 C CNN
-	1    6850 3800
+P 6850 4000
+F 0 "Q1" H 7040 4046 50  0000 L CNN
+F 1 "FGPF7N60RUFD " H 7040 3955 50  0000 L CNN
+F 2 "lib_fp:TO-220-3_Vertical" H 7050 4100 50  0001 C CNN
+F 3 "~" H 6850 4000 50  0001 C CNN
+	1    6850 4000
 	1    0    0    -1
 $EndComp
@@
 L MOSFET-IGBT:R_US R1
 U 1 1 5CDC053C
-P 6300 4000
-F 0 "R1" H 6368 4046 50  0000 L CNN
-F 1 "220" H 6368 3955 50  0000 L CNN
-F 2 "lib_fp:R_Axial_DIN0207_L6.3mm_D2.5mm_P10.16mm_Horizontal" V 6340 3990 50  0001 C CNN
-F 3 "~" H 6300 4000 50  0001 C CNN
-	1    6300 4000
+P 6300 4050
+F 0 "R1" H 6368 4096 50  0000 L CNN
+F 1 "220" H 6368 4005 50  0000 L CNN
+F 2 "lib_fp:R_Axial_DIN0207_L6.3mm_D2.5mm_P10.16mm_Horizontal" V 6340 4040 50  0001 C CNN
+F 3 "~" H 6300 4050 50  0001 C CNN
+	1    6300 4050
 	1    0    0    -1
 $EndComp
@@
 L MOSFET-IGBT:GND #PWR0105
 U 1 1 5CDC0FF3
-P 6950 4400
-F 0 "#PWR0105" H 6950 4150 50  0001 C CNN
-F 1 "GND" H 6955 4227 50  0000 C CNN
-F 2 "" H 6950 4400 50  0001 C CNN
-F 3 "" H 6950 4400 50  0001 C CNN
-	1    6950 4400
+P 4475 4850
+F 0 "#PWR0105" H 4475 4600 50  0001 C CNN
+F 1 "GND" H 4480 4677 50  0000 C CNN
+F 2 "" H 4475 4850 50  0001 C CNN
+F 3 "" H 4475 4850 50  0001 C CNN
+	1    4475 4850
 	1    0    0    -1
 $EndComp
 Wire Wire Line
 	6950 4200 6300 4200
-Wire Wire Line
-	6300 4150 6300 4200
 Connection ~ 6300 4200
 Wire Wire Line
 	6300 4200 5800 4200
 Wire Wire Line
-	6300 3850 6300 3800
+	6300 3900 6300 3800
 Connection ~ 6300 3800
 Wire Wire Line
 	6300 3800 5800 3800
-Wire Wire Line
-	6950 4200 6950 4400
-Wire Wire Line
-	6950 4000 6950 4200
 Connection ~ 6950 4200
 $Comp
 L MOSFET-IGBT:R_US R2
 U 1 1 5CDC3BAC
-P 7550 2850
-F 0 "R2" H 7618 2896 50  0000 L CNN
-F 1 "15" H 7618 2805 50  0000 L CNN
-F 2 "lib_fp:R_Axial_Power_L50.0mm_W9.0mm_P55.88mm" V 7590 2840 50  0001 C CNN
-F 3 "~" H 7550 2850 50  0001 C CNN
-	1    7550 2850
+P 7500 2850
+F 0 "R2" H 7568 2896 50  0000 L CNN
+F 1 "15" H 7568 2805 50  0000 L CNN
+F 2 "lib_fp:R_Axial_Power_L50.0mm_W9.0mm_P55.88mm" V 7540 2840 50  0001 C CNN
+F 3 "~" H 7500 2850 50  0001 C CNN
+	1    7500 2850
 	1    0    0    -1
 $EndComp
@@
 L MOSFET-IGBT:Jumper_NC_Dual JP2
 U 1 1 5CDC4C16
-P 7550 3200
-F 0 "JP2" H 7550 3347 50  0000 C CNN
-F 1 "Jumper_NC_Dual" H 7550 3438 50  0001 C CNN
-F 2 "lib_fp:PinHeader_1x03_P2.54mm_Vertical" H 7550 3200 50  0001 C CNN
-F 3 "~" H 7550 3200 50  0001 C CNN
-	1    7550 3200
+P 7500 3200
+F 0 "JP2" H 7500 3347 50  0000 C CNN
+F 1 "Jumper_NC_Dual" H 7500 3438 50  0001 C CNN
+F 2 "lib_fp:PinHeader_1x03_P2.54mm_Vertical" H 7500 3200 50  0001 C CNN
+F 3 "~" H 7500 3200 50  0001 C CNN
+	1    7500 3200
 	1    0    0    1
 $EndComp
 Wire Wire Line
-	7550 3100 7550 3000
-Wire Wire Line
-	6950 3600 6950 3200
-Wire Wire Line
-	6950 3200 7300 3200
+	7500 3100 7500 3025
+Wire Wire Line
+	6950 3200 7250 3200
 $Comp
 L MOSFET-IGBT:+15V #PWR0106
 U 1 1 5CDC63BE
-P 7550 2600
-F 0 "#PWR0106" H 7550 2450 50  0001 C CNN
-F 1 "+15V" H 7565 2773 50  0000 C CNN
-F 2 "" H 7550 2600 50  0001 C CNN
-F 3 "" H 7550 2600 50  0001 C CNN
-	1    7550 2600
-	1    0    0    -1
-$EndComp
-Wire Wire Line
-	7550 2600 7550 2700
+P 7500 2675
+F 0 "#PWR0106" H 7500 2525 50  0001 C CNN
+F 1 "+15V" H 7515 2848 50  0000 C CNN
+F 2 "" H 7500 2675 50  0001 C CNN
+F 3 "" H 7500 2675 50  0001 C CNN
+	1    7500 2675
+	1    0    0    -1
+$EndComp
+Wire Wire Line
+	7500 2675 7500 2700
 $Comp
 L MOSFET-IGBT:Jumper_NC_Small JP1
 U 1 1 5CDC7EF0
-P 6500 3800
-F 0 "JP1" H 6500 3921 50  0000 C CNN
-F 1 "Jumper_NC_Small" H 6500 3921 50  0001 C CNN
-F 2 "lib_fp:PinHeader_1x02_P2.54mm_Vertical" H 6500 3800 50  0001 C CNN
-F 3 "~" H 6500 3800 50  0001 C CNN
-	1    6500 3800
-	1    0    0    -1
-$EndComp
-Wire Wire Line
-	6400 3800 6300 3800
-Wire Wire Line
-	6650 3800 6600 3800
-Wire Wire Line
-	6300 3800 6300 3550
+P 6650 3900
+F 0 "JP1" V 6650 3800 50  0000 C CNN
+F 1 "Jumper_NC_Small" H 6650 4021 50  0001 C CNN
+F 2 "lib_fp:PinHeader_1x02_P2.54mm_Vertical" H 6650 3900 50  0001 C CNN
+F 3 "~" H 6650 3900 50  0001 C CNN
+	1    6650 3900
+	0    1    1    0
+$EndComp
 $Comp
 L MOSFET-IGBT:IRF8301M Q2
 U 1 1 5CDC9E4F
-P 8000 3800
-F 0 "Q2" H 8206 3846 50  0000 L CNN
-F 1 "IRF840" H 8206 3755 50  0000 L CNN
-F 2 "lib_fp:TO-220-3_Vertical" H 8000 3800 50  0001 C CIN
-F 3 "https://www.infineon.com/dgdl/irf8301mpbf.pdf?fileId=5546d462533600a40153560d0e7a1d58" H 8000 3800 50  0001 L CNN
-	1    8000 3800
-	1    0    0    -1
-$EndComp
-Wire Wire Line
-	8100 3600 8100 3450
-Wire Wire Line
-	8100 3200 7800 3200
-Wire Wire Line
-	6950 4200 8100 4200
-Wire Wire Line
-	8100 4200 8100 4000
+P 7925 4000
+F 0 "Q2" H 8131 4046 50  0000 L CNN
+F 1 "IRF840" H 8131 3955 50  0000 L CNN
+F 2 "lib_fp:TO-220-3_Vertical" H 7925 4000 50  0001 C CIN
+F 3 "https://www.infineon.com/dgdl/irf8301mpbf.pdf?fileId=5546d462533600a40153560d0e7a1d58" H 7925 4000 50  0001 L CNN
+	1    7925 4000
+	1    0    0    -1
+$EndComp
+Wire Wire Line
+	8025 3200 7750 3200
+Wire Wire Line
+	6950 4200 8025 4200
 $Comp
 L MOSFET-IGBT:Jumper_NC_Small JP3
 U 1 1 5CDD2019
-P 7700 3800
-F 0 "JP3" H 7700 3921 50  0000 C CNN
-F 1 "Jumper_NC_Small" H 7700 3921 50  0001 C CNN
-F 2 "lib_fp:PinHeader_1x02_P2.54mm_Vertical" H 7700 3800 50  0001 C CNN
-F 3 "~" H 7700 3800 50  0001 C CNN
-	1    7700 3800
-	1    0    0    -1
-$EndComp
-Wire Wire Line
-	7600 3800 7600 3550
-Wire Wire Line
-	6300 3550 7600 3550
+P 7725 3900
+F 0 "JP3" H 7725 4021 50  0000 C CNN
+F 1 "Jumper_NC_Small" H 7725 4021 50  0001 C CNN
+F 2 "lib_fp:PinHeader_1x02_P2.54mm_Vertical" H 7725 3900 50  0001 C CNN
+F 3 "~" H 7725 3900 50  0001 C CNN
+	1    7725 3900
+	0    1    1    0
+$EndComp
 $Comp
 L MOSFET-IGBT:+15V #PWR0107
@@
 L MOSFET-IGBT:TestPoint_Probe TP3
 U 1 1 5CDF2A14
-P 8100 3450
-F 0 "TP3" H 8253 3551 50  0000 L CNN
-F 1 "TP_VDS" H 8253 3460 50  0000 L CNN
-F 2 "lib_fp:Testpoint" H 8300 3450 50  0001 C CNN
-F 3 "~" H 8300 3450 50  0001 C CNN
-	1    8100 3450
-	1    0    0    -1
-$EndComp
-Connection ~ 8100 3450
-Wire Wire Line
-	8100 3450 8100 3200
+P 7975 3025
+F 0 "TP3" H 8128 3126 50  0000 L CNN
+F 1 "TP_VCE_VDS" H 8128 3035 50  0000 L CNN
+F 2 "lib_fp:Testpoint" H 8175 3025 50  0001 C CNN
+F 3 "~" H 8175 3025 50  0001 C CNN
+	1    7975 3025
+	1    0    0    -1
+$EndComp
 $Comp
 L MOSFET-IGBT:TestPoint_Probe TP1
 U 1 1 5CDF4DF4
-P 6300 3800
-F 0 "TP1" H 6550 3950 50  0000 L CNN
-F 1 "TP_VBE_VGS" H 6450 3850 50  0000 L CNN
-F 2 "lib_fp:Testpoint" H 6500 3800 50  0001 C CNN
-F 3 "~" H 6500 3800 50  0001 C CNN
-	1    6300 3800
+P 6300 3575
+F 0 "TP1" H 6550 3725 50  0000 L CNN
+F 1 "TP_VBE_VGS" H 6450 3625 50  0000 L CNN
+F 2 "lib_fp:Testpoint" H 6500 3575 50  0001 C CNN
+F 3 "~" H 6500 3575 50  0001 C CNN
+	1    6300 3575
 	-1   0    0    -1
 $EndComp
@@
 U 1 1 5CDFA8CD
 P 6950 4200
-F 0 "TP2" H 7102 4301 50  0000 L CNN
-F 1 "GND" H 7102 4210 50  0000 L CNN
+F 0 "TP2" H 7175 4375 50  0000 L CNN
+F 1 "GND" H 7150 4450 50  0000 L CNN
 F 2 "lib_fp:Testpoint" H 7150 4200 50  0001 C CNN
 F 3 "~" H 7150 4200 50  0001 C CNN
 	1    6950 4200
-	1    0    0    -1
+	-1   0    0    1
 $EndComp
 $Comp
@@
 	1    0    0    -1
 $EndComp
+$Comp
+L power:Earth #PWR0104
+U 1 1 5CF247B1
+P 6950 4500
+F 0 "#PWR0104" H 6950 4250 50  0001 C CNN
+F 1 "Earth" H 6950 4350 50  0001 C CNN
+F 2 "" H 6950 4500 50  0001 C CNN
+F 3 "~" H 6950 4500 50  0001 C CNN
+	1    6950 4500
+	1    0    0    -1
+$EndComp
+Wire Wire Line
+	4200 4800 4475 4800
+Connection ~ 4475 4800
+Wire Wire Line
+	4475 4800 4750 4800
+Wire Wire Line
+	7975 3025 7500 3025
+Connection ~ 7500 3025
+Wire Wire Line
+	7500 3025 7500 3000
+Wire Wire Line
+	6300 3800 6650 3800
+Wire Wire Line
+	6950 3800 6950 3200
+Connection ~ 6650 3800
+Wire Wire Line
+	8025 3200 8025 3800
+Wire Wire Line
+	6650 3800 7725 3800
+Wire Wire Line
+	6300 3575 6300 3800
+Wire Wire Line
+	4475 4850 4475 4800
+Wire Wire Line
+	6950 4200 6950 4500
+Text Label 3800 3800 2    50   ~ 0
+PWM_A
+Text Label 3800 4200 2    50   ~ 0
+PWM_B
+Text Notes 5525 4825 0    50   ~ 0
+unir masas
 $EndSCHEMATC
