File: Electronica de Potencia/TP's/TPN3/PCB/Transistores/[Kicad] MOSFET-IGBT/MOSFET-IGBT_PANEL.kicad_pcb (KiCad board)
At the start: 2 copper layers, 247.9 x 177.4 mm, 180 parts, among them J1 Vin, J2 PWM_IN, Q1 FGPF7N60RUFD, Q2 IRF840, T1 50:50

Commit message: Arreglo placa de potencia
Parts:
- removed the D1 at (239.8, 176.2)
- removed the D1 at (150.3, 177.3)
- removed the D1 at (63.6, 178.0)
- removed the D1 at (239.1, 116.3)
- removed the D1 at (150.3, 116.6)
- removed the D1 at (63.2, 118.0)
- removed the D1 at (238.6, 53.2)
- removed the D1 at (150.1, 53.0)
- removed the D1 at (62.8, 52.9)
- removed the D2 at (235.3, 168.6)
- removed the D2 at (145.7, 169.6)
- removed the D2 at (59.0, 170.3)
- removed the D2 at (234.6, 108.7)
- removed the D2 at (145.7, 109.0)
- removed the D2 at (58.6, 110.4)
- removed the D2 at (234.0, 45.6)
- removed the D2 at (145.5, 45.3)
- removed the D2 at (58.2, 45.2)
- removed the D3 at (239.8, 163.0)
- removed the D3 at (150.3, 164.1)
- removed the D3 at (63.6, 164.7)
- removed the D3 at (239.1, 103.1)
- removed the D3 at (150.3, 103.4)
- removed the D3 at (63.2, 104.8)
- removed the D3 at (238.6, 40.0)
- removed the D3 at (150.1, 39.8)
- removed the D3 at (62.8, 39.6)
- removed the D4 at (236.0, 155.4)
- removed the D4 at (146.5, 156.4)
- removed the D4 at (59.8, 157.1)
- removed the D4 at (235.3, 95.5)
- removed the D4 at (146.5, 95.8)
- removed the D4 at (59.4, 97.2)
- removed the D4 at (234.8, 32.4)
- removed the D4 at (146.3, 32.1)
- removed the D4 at (59.0, 32.0)
- removed the G1 at (203.0, 156.7)
- removed the G1 at (113.5, 157.7)
- removed the G1 at (26.7, 158.4)
- removed the G1 at (202.3, 96.7)
- removed the G1 at (113.5, 97.1)
- removed the G1 at (26.4, 98.5)
- removed the G1 at (201.8, 33.7)
- removed the G1 at (113.3, 33.4)
- removed the G1 at (26.0, 33.3)
- removed the HS1 at (280.2, 141.7)
- removed the HS1 at (190.7, 142.7)
- removed the HS1 at (104.0, 143.4)
- removed the HS1 at (279.5, 81.8)
- removed the HS1 at (190.7, 82.1)
- removed the HS1 at (103.6, 83.5)
- removed the HS1 at (279.0, 18.7)
- removed the HS1 at (190.5, 18.4)
- removed the HS1 at (103.2, 18.3)
- removed the HS2 at (280.6, 164.0)
- removed the HS2 at (191.1, 165.1)
- removed the HS2 at (104.3, 165.8)
- removed the HS2 at (279.9, 104.1)
- removed the HS2 at (191.1, 104.4)
- removed the HS2 at (104.0, 105.8)
- removed the HS2 at (279.4, 41.0)
- removed the HS2 at (190.9, 40.8)
- removed the HS2 at (103.6, 40.7)
- removed the J1 at (201.2, 144.7)
- removed the J1 at (111.7, 145.8)
- removed the J1 at (25.0, 146.5)
- removed the J1 at (200.5, 84.8)
- removed the J1 at (111.7, 85.1)
- removed the J1 at (24.6, 86.5)
- removed the J1 at (200.0, 21.7)
- removed the J1 at (111.5, 21.5)
- removed the J1 at (24.2, 21.4)
- removed the J2 at (203.0, 164.3)
- removed the J2 at (113.5, 165.3)
- removed the J2 at (26.7, 166.0)
- removed the J2 at (202.3, 104.4)
- removed the J2 at (113.5, 104.7)
- removed the J2 at (26.4, 106.1)
- removed the J2 at (201.8, 41.3)
- removed the J2 at (113.3, 41.0)
- removed the J2 at (26.0, 40.9)
- removed the JP1 at (248.7, 162.8)
- removed the JP1 at (159.2, 163.8)
- removed the JP1 at (72.5, 164.5)
- removed the JP1 at (248.0, 102.8)
- removed the JP1 at (159.2, 103.2)
- removed the JP1 at (72.1, 104.6)
- removed the JP1 at (247.5, 39.8)
- removed the JP1 at (159.0, 39.5)
- removed the JP1 at (71.7, 39.4)
- removed the JP2 at (248.7, 171.7)
- removed the JP2 at (159.2, 172.7)
- removed the JP2 at (72.5, 173.4)
- removed the JP2 at (248.0, 111.7)
- removed the JP2 at (159.2, 112.1)
- removed the JP2 at (72.1, 113.5)
- removed the JP2 at (247.5, 48.7)
- removed the JP2 at (159.0, 48.4)
- removed the JP2 at (71.7, 48.3)
- removed the JP3 at (248.7, 154.6)
- removed the JP3 at (159.2, 155.7)
- removed the JP3 at (72.5, 156.4)
- removed the JP3 at (248.0, 94.7)
- removed the JP3 at (159.2, 95.0)
- removed the JP3 at (72.1, 96.4)
- removed the JP3 at (247.5, 31.6)
- removed the JP3 at (159.0, 31.4)
- removed the JP3 at (71.7, 31.3)
- removed the Q1 at (257.2, 171.3)
- removed the Q1 at (167.7, 172.3)
- removed the Q1 at (81.0, 173.0)
- removed the Q1 at (256.5, 111.4)
- removed the Q1 at (167.7, 111.7)
- removed the Q1 at (80.6, 113.1)
- removed the Q1 at (256.0, 48.3)
- removed the Q1 at (167.5, 48.0)
- removed the Q1 at (80.2, 47.9)
- removed the Q2 at (256.7, 149.0)
- removed the Q2 at (167.2, 150.1)
- removed the Q2 at (80.5, 150.8)
- removed the Q2 at (256.0, 89.1)
- removed the Q2 at (167.2, 89.5)
- removed the Q2 at (80.1, 90.9)
- removed the Q2 at (255.5, 26.1)
- removed the Q2 at (167.0, 25.8)
- removed the Q2 at (79.7, 25.7)
- removed the R1 at (232.2, 151.6)
- removed the R1 at (142.7, 152.6)
- removed the R1 at (56.0, 153.3)
- removed the R1 at (231.5, 91.7)
- removed the R1 at (142.7, 92.0)
- removed the R1 at (55.6, 93.4)
- removed the R1 at (231.0, 28.6)
- removed the R1 at (142.5, 28.3)
- removed the R1 at (55.2, 28.2)
- removed the R2 at (201.7, 184.6)
- removed the R2 at (112.2, 185.6)
- removed the R2 at (25.5, 186.3)
- removed the R2 at (201.0, 124.7)
- removed the R2 at (112.2, 125.0)
- removed the R2 at (25.1, 126.4)
- removed the R2 at (200.5, 61.6)
- removed the R2 at (112.0, 61.3)
- removed the R2 at (24.7, 61.2)
- removed the T1 at (230.9, 149.0)
- removed the T1 at (141.4, 150.1)
- removed the T1 at (54.7, 150.8)
- removed the T1 at (230.3, 89.1)
- removed the T1 at (141.4, 89.5)
- removed the T1 at (54.3, 90.9)
- removed the T1 at (229.7, 26.1)
- removed the T1 at (141.2, 25.8)
- removed the T1 at (53.9, 25.7)
- removed the TP1 at (217.5, 142.4)
- removed the TP1 at (128.0, 143.5)
- removed the TP1 at (41.2, 144.2)
- removed the TP1 at (216.8, 82.5)
- removed the TP1 at (128.0, 82.9)
- removed the TP1 at (40.9, 84.3)
- removed the TP1 at (216.3, 19.5)
- removed the TP1 at (127.7, 19.2)
- removed the TP1 at (40.4, 19.1)
- removed the TP2 at (235.3, 142.4)
- removed the TP2 at (145.7, 143.5)
- removed the TP2 at (59.0, 144.2)
- removed the TP2 at (234.6, 82.5)
- removed the TP2 at (145.7, 82.9)
- removed the TP2 at (58.6, 84.3)
- removed the TP2 at (234.0, 19.5)
- removed the TP2 at (145.5, 19.2)
- removed the TP2 at (58.2, 19.1)
- removed the TP3 at (253.0, 142.4)
- removed the TP3 at (163.5, 143.5)
- removed the TP3 at (76.8, 144.2)
- removed the TP3 at (252.3, 82.5)
- removed the TP3 at (163.5, 82.9)
- removed the TP3 at (76.4, 84.3)
- removed the TP3 at (251.8, 19.5)
- removed the TP3 at (163.3, 19.2)
- removed the TP3 at (76.0, 19.1)
- added D1: 1N4148, lib_fp:D_DO-34_SOD68_P7.62mm_Horizontal, F.Cu at (233.4, 162.9)
- added D1: 1N4148, lib_fp:D_DO-34_SOD68_P7.62mm_Horizontal, F.Cu at (146.9, 163.0)
- added D1: 1N4148, lib_fp:D_DO-34_SOD68_P7.62mm_Horizontal, F.Cu at (59.6, 163.0)
- added D1: 1N4148, lib_fp:D_DO-34_SOD68_P7.62mm_Horizontal, F.Cu at (233.1, 105.4)
- added D1: 1N4148, lib_fp:D_DO-34_SOD68_P7.62mm_Horizontal, F.Cu at (146.6, 105.5)
- added D1: 1N4148, lib_fp:D_DO-34_SOD68_P7.62mm_Horizontal, F.Cu at (59.3, 105.5)
- added D1: 1N4148, lib_fp:D_DO-34_SOD68_P7.62mm_Horizontal, F.Cu at (233.5, 39.8)
- added D1: 1N4148, lib_fp:D_DO-34_SOD68_P7.62mm_Horizontal, F.Cu at (147.0, 39.9)
- added D1: 1N4148, lib_fp:D_DO-34_SOD68_P7.62mm_Horizontal, F.Cu at (59.7, 40.0)
- added D2: 1N4148, lib_fp:D_DO-34_SOD68_P7.62mm_Horizontal, F.Cu at (225.8, 158.7)
- added D2: 1N4148, lib_fp:D_DO-34_SOD68_P7.62mm_Horizontal, F.Cu at (139.3, 158.8)
- added D2: 1N4148, lib_fp:D_DO-34_SOD68_P7.62mm_Horizontal, F.Cu at (52.0, 158.8)
- added D2: 1N4148, lib_fp:D_DO-34_SOD68_P7.62mm_Horizontal, F.Cu at (225.5, 101.2)
- added D2: 1N4148, lib_fp:D_DO-34_SOD68_P7.62mm_Horizontal, F.Cu at (139.0, 101.3)
- added D2: 1N4148, lib_fp:D_DO-34_SOD68_P7.62mm_Horizontal, F.Cu at (51.7, 101.4)
- added D2: 1N4148, lib_fp:D_DO-34_SOD68_P7.62mm_Horizontal, F.Cu at (225.9, 35.6)
- added D2: 1N4148, lib_fp:D_DO-34_SOD68_P7.62mm_Horizontal, F.Cu at (139.4, 35.8)
- added D2: 1N4148, lib_fp:D_DO-34_SOD68_P7.62mm_Horizontal, F.Cu at (52.1, 35.8)
- added D3: 1N4148, lib_fp:D_DO-34_SOD68_P7.62mm_Horizontal, F.Cu at (233.3, 168.0)
- added D3: 1N4148, lib_fp:D_DO-34_SOD68_P7.62mm_Horizontal, F.Cu at (146.7, 168.1)
- added D3: 1N4148, lib_fp:D_DO-34_SOD68_P7.62mm_Horizontal, F.Cu at (59.4, 168.2)
- added D3: 1N4148, lib_fp:D_DO-34_SOD68_P7.62mm_Horizontal, F.Cu at (233.0, 110.5)
- added D3: 1N4148, lib_fp:D_DO-34_SOD68_P7.62mm_Horizontal, F.Cu at (146.4, 110.7)
- added D3: 1N4148, lib_fp:D_DO-34_SOD68_P7.62mm_Horizontal, F.Cu at (59.1, 110.7)
- added D3: 1N4148, lib_fp:D_DO-34_SOD68_P7.62mm_Horizontal, F.Cu at (233.4, 45.0)
- added D3: 1N4148, lib_fp:D_DO-34_SOD68_P7.62mm_Horizontal, F.Cu at (146.9, 45.1)
- added D3: 1N4148, lib_fp:D_DO-34_SOD68_P7.62mm_Horizontal, F.Cu at (59.6, 45.1)
- added D4: 1N4148, lib_fp:D_DO-34_SOD68_P7.62mm_Horizontal, F.Cu at (225.8, 172.4)
- added D4: 1N4148, lib_fp:D_DO-34_SOD68_P7.62mm_Horizontal, F.Cu at (139.3, 172.5)
- added D4: 1N4148, lib_fp:D_DO-34_SOD68_P7.62mm_Horizontal, F.Cu at (52.0, 172.5)
- added D4: 1N4148, lib_fp:D_DO-34_SOD68_P7.62mm_Horizontal, F.Cu at (225.5, 114.9)
- added D4: 1N4148, lib_fp:D_DO-34_SOD68_P7.62mm_Horizontal, F.Cu at (139.0, 115.0)
- added D4: 1N4148, lib_fp:D_DO-34_SOD68_P7.62mm_Horizontal, F.Cu at (51.7, 115.0)
- added D4: 1N4148, lib_fp:D_DO-34_SOD68_P7.62mm_Horizontal, F.Cu at (225.9, 49.3)
- added D4: 1N4148, lib_fp:D_DO-34_SOD68_P7.62mm_Horizontal, F.Cu at (139.4, 49.4)
- added D4: 1N4148, lib_fp:D_DO-34_SOD68_P7.62mm_Horizontal, F.Cu at (52.1, 49.5)
- added G1: logo, lib_fp:logo_utn_fsilk_small, F.Cu at (195.6, 154.1)
- added G1: logo, lib_fp:logo_utn_fsilk_small, F.Cu at (109.1, 154.2)
- added G1: logo, lib_fp:logo_utn_fsilk_small, F.Cu at (21.8, 154.3)
- added G1: logo, lib_fp:logo_utn_fsilk_small, F.Cu at (195.3, 96.6)
- added G1: logo, lib_fp:logo_utn_fsilk_small, F.Cu at (108.8, 96.8)
- added G1: logo, lib_fp:logo_utn_fsilk_small, F.Cu at (21.5, 96.8)
- added G1: logo, lib_fp:logo_utn_fsilk_small, F.Cu at (195.8, 31.1)
- added G1: logo, lib_fp:logo_utn_fsilk_small, F.Cu at (109.2, 31.2)
- added G1: logo, lib_fp:logo_utn_fsilk_small, F.Cu at (21.9, 31.2)
- added HS1: Heatsink, lib_fp:Heatsink_TO220_A, F.Cu at (272.6, 141.1)
- added HS1: Heatsink, lib_fp:Heatsink_TO220_A, F.Cu at (186.1, 141.3)
- added HS1: Heatsink, lib_fp:Heatsink_TO220_A, F.Cu at (98.7, 141.3)
- added HS1: Heatsink, lib_fp:Heatsink_TO220_A, F.Cu at (272.3, 83.7)
- added HS1: Heatsink, lib_fp:Heatsink_TO220_A, F.Cu at (185.8, 83.8)
- added HS1: Heatsink, lib_fp:Heatsink_TO220_A, F.Cu at (98.4, 83.8)
- added HS1: Heatsink, lib_fp:Heatsink_TO220_A, F.Cu at (272.7, 18.1)
- added HS1: Heatsink, lib_fp:Heatsink_TO220_A, F.Cu at (186.2, 18.2)
- added HS1: Heatsink, lib_fp:Heatsink_TO220_A, F.Cu at (98.9, 18.3)
- added HS2: Heatsink, lib_fp:Heatsink_TO220_A, F.Cu at (272.9, 163.5)
- added HS2: Heatsink, lib_fp:Heatsink_TO220_A, F.Cu at (186.4, 163.6)
- added HS2: Heatsink, lib_fp:Heatsink_TO220_A, F.Cu at (99.1, 163.7)
- added HS2: Heatsink, lib_fp:Heatsink_TO220_A, F.Cu at (272.6, 106.0)
- added HS2: Heatsink, lib_fp:Heatsink_TO220_A, F.Cu at (186.1, 106.1)
- added HS2: Heatsink, lib_fp:Heatsink_TO220_A, F.Cu at (98.8, 106.2)
- added HS2: Heatsink, lib_fp:Heatsink_TO220_A, F.Cu at (273.1, 40.5)
- added HS2: Heatsink, lib_fp:Heatsink_TO220_A, F.Cu at (186.6, 40.6)
- added HS2: Heatsink, lib_fp:Heatsink_TO220_A, F.Cu at (99.2, 40.6)
- added J1: Vin, lib_fp:TerminalBlock_bornier-2_P5.08mm, F.Cu at (193.6, 144.2)
- added J1: Vin, lib_fp:TerminalBlock_bornier-2_P5.08mm, F.Cu at (107.1, 144.3)
- added J1: Vin, lib_fp:TerminalBlock_bornier-2_P5.08mm, F.Cu at (19.7, 144.4)
- added J1: Vin, lib_fp:TerminalBlock_bornier-2_P5.08mm, F.Cu at (193.3, 86.7)
- added J1: Vin, lib_fp:TerminalBlock_bornier-2_P5.08mm, F.Cu at (106.8, 86.8)
- added J1: Vin, lib_fp:TerminalBlock_bornier-2_P5.08mm, F.Cu at (19.4, 86.9)
- added J1: Vin, lib_fp:TerminalBlock_bornier-2_P5.08mm, F.Cu at (193.7, 21.2)
- added J1: Vin, lib_fp:TerminalBlock_bornier-2_P5.08mm, F.Cu at (107.2, 21.3)
- added J1: Vin, lib_fp:TerminalBlock_bornier-2_P5.08mm, F.Cu at (19.9, 21.3)
- added J2: PWM_IN, lib_fp:TerminalBlock_bornier-3_P5.08mm, F.Cu at (197.5, 163.7)
- added J2: PWM_IN, lib_fp:TerminalBlock_bornier-3_P5.08mm, F.Cu at (111.0, 163.8)
- added J2: PWM_IN, lib_fp:TerminalBlock_bornier-3_P5.08mm, F.Cu at (23.7, 163.9)
- added J2: PWM_IN, lib_fp:TerminalBlock_bornier-3_P5.08mm, F.Cu at (197.2, 106.2)
- added J2: PWM_IN, lib_fp:TerminalBlock_bornier-3_P5.08mm, F.Cu at (110.7, 106.3)
- added J2: PWM_IN, lib_fp:TerminalBlock_bornier-3_P5.08mm, F.Cu at (23.3, 106.4)
- added J2: PWM_IN, lib_fp:TerminalBlock_bornier-3_P5.08mm, F.Cu at (197.6, 40.7)
- added J2: PWM_IN, lib_fp:TerminalBlock_bornier-3_P5.08mm, F.Cu at (111.1, 40.8)
- added J2: PWM_IN, lib_fp:TerminalBlock_bornier-3_P5.08mm, F.Cu at (23.8, 40.8)
- added JP1: Jumper_NC_Small, lib_fp:PinHeader_1x02_P2.54mm_Vertical, F.Cu at (242.0, 158.6)
- added JP1: Jumper_NC_Small, lib_fp:PinHeader_1x02_P2.54mm_Vertical, F.Cu at (68.2, 158.8)
- added JP1: Jumper_NC_Small, lib_fp:PinHeader_1x02_P2.54mm_Vertical, F.Cu at (155.5, 158.7)
- added JP1: Jumper_NC_Small, lib_fp:PinHeader_1x02_P2.54mm_Vertical, F.Cu at (241.7, 101.1)
- added JP1: Jumper_NC_Small, lib_fp:PinHeader_1x02_P2.54mm_Vertical, F.Cu at (67.9, 101.3)
- added JP1: Jumper_NC_Small, lib_fp:PinHeader_1x02_P2.54mm_Vertical, F.Cu at (155.2, 101.3)
- added JP1: Jumper_NC_Small, lib_fp:PinHeader_1x02_P2.54mm_Vertical, F.Cu at (242.1, 35.6)
- added JP1: Jumper_NC_Small, lib_fp:PinHeader_1x02_P2.54mm_Vertical, F.Cu at (155.6, 35.7)
- added JP1: Jumper_NC_Small, lib_fp:PinHeader_1x02_P2.54mm_Vertical, F.Cu at (68.3, 35.7)
- added JP2: Jumper_NC_Dual, lib_fp:PinHeader_1x03_P2.54mm_Vertical, F.Cu at (242.4, 168.6)
- added JP2: Jumper_NC_Dual, lib_fp:PinHeader_1x03_P2.54mm_Vertical, F.Cu at (68.6, 168.7)
- added JP2: Jumper_NC_Dual, lib_fp:PinHeader_1x03_P2.54mm_Vertical, F.Cu at (155.9, 168.7)
- added JP2: Jumper_NC_Dual, lib_fp:PinHeader_1x03_P2.54mm_Vertical, F.Cu at (242.1, 111.1)
- added JP2: Jumper_NC_Dual, lib_fp:PinHeader_1x03_P2.54mm_Vertical, F.Cu at (68.3, 111.2)
- added JP2: Jumper_NC_Dual, lib_fp:PinHeader_1x03_P2.54mm_Vertical, F.Cu at (155.6, 111.2)
- added JP2: Jumper_NC_Dual, lib_fp:PinHeader_1x03_P2.54mm_Vertical, F.Cu at (242.6, 45.5)
- added JP2: Jumper_NC_Dual, lib_fp:PinHeader_1x03_P2.54mm_Vertical, F.Cu at (156.1, 45.6)
- added JP2: Jumper_NC_Dual, lib_fp:PinHeader_1x03_P2.54mm_Vertical, F.Cu at (68.7, 45.7)
- added JP3: Jumper_NC_Small, lib_fp:PinHeader_1x02_P2.54mm_Vertical, F.Cu at (241.9, 153.6)
- added JP3: Jumper_NC_Small, lib_fp:PinHeader_1x02_P2.54mm_Vertical, F.Cu at (155.4, 153.7)
- added JP3: Jumper_NC_Small, lib_fp:PinHeader_1x02_P2.54mm_Vertical, F.Cu at (68.1, 153.8)
- added JP3: Jumper_NC_Small, lib_fp:PinHeader_1x02_P2.54mm_Vertical, F.Cu at (241.6, 96.1)
- added JP3: Jumper_NC_Small, lib_fp:PinHeader_1x02_P2.54mm_Vertical, F.Cu at (155.1, 96.3)
- added JP3: Jumper_NC_Small, lib_fp:PinHeader_1x02_P2.54mm_Vertical, F.Cu at (67.8, 96.3)
- added JP3: Jumper_NC_Small, lib_fp:PinHeader_1x02_P2.54mm_Vertical, F.Cu at (242.0, 30.6)
- added JP3: Jumper_NC_Small, lib_fp:PinHeader_1x02_P2.54mm_Vertical, F.Cu at (155.5, 30.7)
- added JP3: Jumper_NC_Small, lib_fp:PinHeader_1x02_P2.54mm_Vertical, F.Cu at (68.2, 30.7)
- added Q1: FGPF7N60RUFD, lib_fp:TO-220-3_Vertical, F.Cu at (249.6, 170.7)
- added Q1: FGPF7N60RUFD, lib_fp:TO-220-3_Vertical, F.Cu at (163.1, 170.9)
- added Q1: FGPF7N60RUFD, lib_fp:TO-220-3_Vertical, F.Cu at (75.7, 170.9)
- added Q1: FGPF7N60RUFD, lib_fp:TO-220-3_Vertical, F.Cu at (249.3, 113.3)
- added Q1: FGPF7N60RUFD, lib_fp:TO-220-3_Vertical, F.Cu at (162.8, 113.4)
- added Q1: FGPF7N60RUFD, lib_fp:TO-220-3_Vertical, F.Cu at (75.4, 113.4)
- added Q1: FGPF7N60RUFD, lib_fp:TO-220-3_Vertical, F.Cu at (249.7, 47.7)
- added Q1: FGPF7N60RUFD, lib_fp:TO-220-3_Vertical, F.Cu at (163.2, 47.8)
- added Q1: FGPF7N60RUFD, lib_fp:TO-220-3_Vertical, F.Cu at (75.9, 47.9)
- added Q2: IRF840, lib_fp:TO-220-3_Vertical, F.Cu at (249.1, 148.5)
- added Q2: IRF840, lib_fp:TO-220-3_Vertical, F.Cu at (162.6, 148.6)
- added Q2: IRF840, lib_fp:TO-220-3_Vertical, F.Cu at (75.2, 148.7)
- added Q2: IRF840, lib_fp:TO-220-3_Vertical, F.Cu at (248.8, 91.0)
- added Q2: IRF840, lib_fp:TO-220-3_Vertical, F.Cu at (162.3, 91.2)
- added Q2: IRF840, lib_fp:TO-220-3_Vertical, F.Cu at (74.9, 91.2)
- added Q2: IRF840, lib_fp:TO-220-3_Vertical, F.Cu at (249.2, 25.5)
- added Q2: IRF840, lib_fp:TO-220-3_Vertical, F.Cu at (162.7, 25.6)
- added Q2: IRF840, lib_fp:TO-220-3_Vertical, F.Cu at (75.4, 25.6)
- added R1: 220, lib_fp:R_Axial_DIN0207_L6.3mm_D2.5mm_P10.16mm_Horizontal, F.Cu at (226.1, 152.8)
- added R1: 220, lib_fp:R_Axial_DIN0207_L6.3mm_D2.5mm_P10.16mm_Horizontal, F.Cu at (139.6, 152.9)
- added R1: 220, lib_fp:R_Axial_DIN0207_L6.3mm_D2.5mm_P10.16mm_Horizontal, F.Cu at (52.3, 152.9)
- added R1: 220, lib_fp:R_Axial_DIN0207_L6.3mm_D2.5mm_P10.16mm_Horizontal, F.Cu at (225.8, 95.3)
- added R1: 220, lib_fp:R_Axial_DIN0207_L6.3mm_D2.5mm_P10.16mm_Horizontal, F.Cu at (139.3, 95.4)
- added R1: 220, lib_fp:R_Axial_DIN0207_L6.3mm_D2.5mm_P10.16mm_Horizontal, F.Cu at (52.0, 95.5)
- added R1: 220, lib_fp:R_Axial_DIN0207_L6.3mm_D2.5mm_P10.16mm_Horizontal, F.Cu at (226.3, 29.7)
- added R1: 220, lib_fp:R_Axial_DIN0207_L6.3mm_D2.5mm_P10.16mm_Horizontal, F.Cu at (139.8, 29.9)
- added R1: 220, lib_fp:R_Axial_DIN0207_L6.3mm_D2.5mm_P10.16mm_Horizontal, F.Cu at (52.4, 29.9)
- added R2: 15, lib_fp:R_Axial_Power_L50.0mm_W9.0mm_P55.88mm, F.Cu at (194.1, 184.1)
- added R2: 15, lib_fp:R_Axial_Power_L50.0mm_W9.0mm_P55.88mm, F.Cu at (20.2, 184.2)
- added R2: 15, lib_fp:R_Axial_Power_L50.0mm_W9.0mm_P55.88mm, F.Cu at (107.6, 184.2)
- added R2: 15, lib_fp:R_Axial_Power_L50.0mm_W9.0mm_P55.88mm, F.Cu at (193.8, 126.6)
- added R2: 15, lib_fp:R_Axial_Power_L50.0mm_W9.0mm_P55.88mm, F.Cu at (19.9, 126.8)
- added R2: 15, lib_fp:R_Axial_Power_L50.0mm_W9.0mm_P55.88mm, F.Cu at (107.3, 126.7)
- added R2: 15, lib_fp:R_Axial_Power_L50.0mm_W9.0mm_P55.88mm, F.Cu at (194.2, 61.0)
- added R2: 15, lib_fp:R_Axial_Power_L50.0mm_W9.0mm_P55.88mm, F.Cu at (107.7, 61.2)
- added R2: 15, lib_fp:R_Axial_Power_L50.0mm_W9.0mm_P55.88mm, F.Cu at (20.4, 61.2)
- added T1: 50:50, lib_fp:Transformador_EE25, F.Cu at (201.3, 177.1)
- added T1: 50:50, lib_fp:Transformador_EE25, F.Cu at (114.8, 177.2)
- added T1: 50:50, lib_fp:Transformador_EE25, F.Cu at (27.5, 177.3)
- added T1: 50:50, lib_fp:Transformador_EE25, F.Cu at (201.0, 119.6)
- added T1: 50:50, lib_fp:Transformador_EE25, F.Cu at (114.5, 119.7)
- added T1: 50:50, lib_fp:Transformador_EE25, F.Cu at (27.2, 119.8)
- added T1: 50:50, lib_fp:Transformador_EE25, F.Cu at (201.4, 54.1)
- added T1: 50:50, lib_fp:Transformador_EE25, F.Cu at (114.9, 54.2)
- added T1: 50:50, lib_fp:Transformador_EE25, F.Cu at (27.6, 54.2)
- added TP1: TP_VBE_VGS, lib_fp:Testpoint, F.Cu at (208.7, 142.2)
- added TP1: TP_VBE_VGS, lib_fp:Testpoint, F.Cu at (34.9, 142.4)
- added TP1: TP_VBE_VGS, lib_fp:Testpoint, F.Cu at (122.2, 142.3)
- added TP1: TP_VBE_VGS, lib_fp:Testpoint, F.Cu at (208.4, 84.7)
- added TP1: TP_VBE_VGS, lib_fp:Testpoint, F.Cu at (34.6, 84.9)
- added TP1: TP_VBE_VGS, lib_fp:Testpoint, F.Cu at (121.9, 84.9)
- added TP1: TP_VBE_VGS, lib_fp:Testpoint, F.Cu at (208.8, 19.2)
- added TP1: TP_VBE_VGS, lib_fp:Testpoint, F.Cu at (122.3, 19.3)
- added TP1: TP_VBE_VGS, lib_fp:Testpoint, F.Cu at (35.0, 19.3)
- added TP2: GND, lib_fp:Testpoint, F.Cu at (227.7, 142.2)
- added TP2: GND, lib_fp:Testpoint, F.Cu at (53.9, 142.4)
- added TP2: GND, lib_fp:Testpoint, F.Cu at (141.2, 142.3)
- added TP2: GND, lib_fp:Testpoint, F.Cu at (227.4, 84.7)
- added TP2: GND, lib_fp:Testpoint, F.Cu at (53.6, 84.9)
- added TP2: GND, lib_fp:Testpoint, F.Cu at (140.9, 84.9)
- added TP2: GND, lib_fp:Testpoint, F.Cu at (227.8, 19.2)
- added TP2: GND, lib_fp:Testpoint, F.Cu at (141.3, 19.3)
- added TP2: GND, lib_fp:Testpoint, F.Cu at (54.0, 19.3)
- added TP3: TP_VCE_VDS, lib_fp:Testpoint, F.Cu at (245.9, 142.2)
- added TP3: TP_VCE_VDS, lib_fp:Testpoint, F.Cu at (72.1, 142.3)
- added TP3: TP_VCE_VDS, lib_fp:Testpoint, F.Cu at (159.4, 142.3)
- added TP3: TP_VCE_VDS, lib_fp:Testpoint, F.Cu at (245.6, 84.7)
- added TP3: TP_VCE_VDS, lib_fp:Testpoint, F.Cu at (71.8, 84.8)
- added TP3: TP_VCE_VDS, lib_fp:Testpoint, F.Cu at (159.1, 84.8)
- added TP3: TP_VCE_VDS, lib_fp:Testpoint, F.Cu at (246.1, 19.1)
- added TP3: TP_VCE_VDS, lib_fp:Testpoint, F.Cu at (159.6, 19.2)
- added TP3: TP_VCE_VDS, lib_fp:Testpoint, F.Cu at (72.2, 19.3)
Routing:
- net (no net): track 3600.3 -> 5545.8 mm, vias 18 -> 16
- net GND: track 0.00 -> 109.6 mm
- net +15V: track 0.00 -> 109.3 mm
- net Earth: track 0.00 -> 96.4 mm, vias 0 -> 2
- net Net-(JP1-Pad1): track 0.00 -> 93.9 mm
- net Net-(JP2-Pad2): track 0.00 -> 83.1 mm
- net /PWM_B: track 0.00 -> 63.2 mm
- net Net-(JP2-Pad3): track 0.00 -> 53.8 mm
- net /PWM_A: track 0.00 -> 48.6 mm
- net Net-(JP1-Pad2): track 0.00 -> 16.0 mm
- net Net-(JP2-Pad1): track 0.00 -> 12.0 mm
- net Net-(JP3-Pad2): track 0.00 -> 7.19 mm
- added copper zone on B.Cu, net GND
Other:
- board size 247.9 x 177.4 mm -> 245.1 x 175.5 mm
