File: Electronica de Potencia/TP's/TPN5/[KiCad] PCB/Fuente/Fuente.kicad_pcb (KiCad board)
At the start: 2 copper layers, 145 x 150.1 mm, 76 parts, among them J1 220 VAC, J2 Entrada +20 V, J3 Main_OUT, J4 Main_IN, J5 Ctrl_OUT, J6 Ctrl_IN, J7 Salida +24V, Q1 IRF840, Q2 IRF840, SW1 ROCKER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

Commit message: Actualizo desde Envy
Other:
- net class Default: clearance 0.8 -> 0.4
- rule trace_clearance: 0.8 -> 0.4
Changed lines of the file:
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@@
-(kicad_pcb (version 20171130) (host pcbnew "(5.0.1)-4")
+(kicad_pcb (version 20171130) (host pcbnew 5.1.4)
   (general
     (thickness 1.6)
@@
     (user_trace_width 4)
     (user_trace_width 5)
-    (trace_clearance 0.8)
+    (trace_clearance 0.4)
     (zone_clearance 1)
     (zone_45_only no)
     (trace_min 0.4)
-    (segment_width 0.2)
-    (edge_width 0.05)
     (via_size 1.5)
     (via_drill 1)
@@
     (uvia_min_size 0.2)
     (uvia_min_drill 0.1)
+    (edge_width 0.05)
+    (segment_width 0.2)
     (pcb_text_width 0.3)
     (pcb_text_size 1.5 1.5)
@@
     (aux_axis_origin 16.647 17.172)
     (grid_origin 216.274 87.037)
-    (visible_elements 7FFFFFFF)
+    (visible_elements FFFFFF7F)
     (pcbplotparams
       (layerselection 0x010fc_ffffffff)
@@
   (net 53 "Net-(C17-Pad1)")
   (net_class Default "Esta es la clase de red por defecto."
-    (clearance 0.8)
+    (clearance 0.4)
     (trace_width 1.2)
     (via_dia 1.5)
@@
     (uvia_dia 0.3)
     (uvia_drill 0.1)
+    (diff_pair_width 0.8)
     (diff_pair_gap 0.25)
-    (diff_pair_width 0.8)
     (add_net F)
     (add_net GNDPWR)
